File: DMM_KiCAD_V3_next KiCAD9/DMM_KiCAD_V3_next KiCAD9.kicad_pcb (KiCad board)
At the start: 4 copper layers, 68.5 x 53.2 mm, 78 parts, among them J1 Conn_01x07_Pin, J10 ANALOG, J11 I_Input, J12 Conn_01x02_Pin, J13 DIGITAL1, J14 Barrel_Jack, J15 Barrel_Jack, J16 Conn_01x01_Socket, J17 Conn_01x01_Socket, J2 MicoSD, J3 Conn_01x07_Pin, J4 IR Connection, J5 POWER2, J6 POWER1, J7 Conn_01x02_Pin, J8 DIGITAL2, J9 Out to Screen, Q1 MMBT3904, Q2 SI2302 MOSFET, Q3 MMBT3904, Q4 MMBT3904, Q5 MMBT3904, Q6 BSS138, Q7 BSS138, SW1 SW_Push, SW2 SW_Push, SW3 SW_SPDT, SW4 SW_Push, U1 LM317_TO-220, U10 LM4040DBZ-2.5, U11 LM4040DBZ-5, U3 ADS1115IDGS, U7 MAX1683, U9 TPS613222ADBV

Commit message: Mostly working on the next PCB
Parts:
- removed C1: 0.47uF, Capacitor_SMD:C_0805_2012Metric_Pad1.18x1.45mm_HandSolder
- removed C14: 2.2uF, Capacitor_SMD:C_0805_2012Metric_Pad1.18x1.45mm_HandSolder
- removed Q3, Q4, Q5: MMBT3904, Package_TO_SOT_SMD:SOT-23
- removed R10, R11, R19, R20: 10K, Resistor_SMD:R_0805_2012Metric_Pad1.20x1.40mm_HandSolder
- removed R12: 75K, Resistor_SMD:R_0805_2012Metric_Pad1.20x1.40mm_HandSolder
- removed R13, R15, R16, R25, R26: 1K, Resistor_SMD:R_0805_2012Metric_Pad1.20x1.40mm_HandSolder
- removed R7: 22K, Resistor_SMD:R_0805_2012Metric_Pad1.20x1.40mm_HandSolder
- removed R8: 4.7K, Resistor_SMD:R_0805_2012Metric_Pad1.20x1.40mm_HandSolder
- added Q8: SI2302 MOSFET, Package_TO_SOT_SMD:SOT-23, F.Cu at (161.6, 83.5)
- added R24: 1.0M, Resistor_SMD:R_0805_2012Metric_Pad1.20x1.40mm_HandSolder, F.Cu at (161.6, 86.8)
- added RN1: R_Pack04_SIP, Resistor_SMD:R_Array_Convex_4x1206, F.Cu at (132.4, 65.4)
- added RN2: R_Pack04_SIP, Resistor_SMD:R_Array_Convex_4x1206, F.Cu at (122.6, 107.0)
- added U2: ~, Package_SO:SOIC-8_3.9x4.9mm_P1.27mm, F.Cu at (121.9, 61.0)
- added U4: ~, Package_SO:SOIC-8_3.9x4.9mm_P1.27mm, F.Cu at (105.4, 91.4)
- moved R27 2.03 mm to (123.2, 89.9)
- moved Q2 0.37 mm to (120.7, 68.6)
- moved C18 0.13 mm to (124.5, 67.9)
Connections:
- J1 pad 3: +3V3 -> SDA
- J2 pad 6: +3V3 -> SDA
- J6 pad 4: +3V3 -> SDA
- Q6 pad 1: +3V3 -> SDA
- Q7 pad 1: +3V3 -> SDA
- U1 pad 3: Net-(Q5-E) -> /Driver_U2_Out_B
Routing:
- net +3V3: track 67.4 -> 0.00 mm, vias 2 -> 0
- net SDA: track 69.8 -> 137.1 mm, vias 3 -> 7
- net +9V: track 34.1 -> 53.5 mm
- net D5~ (IR): track 59.8 -> 77.0 mm, vias 0 -> 2
- net Net-(Q4-C): track 8.99 -> 0.00 mm
- net Net-(Q5-E): track 8.88 -> 0.00 mm
- net /V Ref to ADS: track 31.8 -> 23.5 mm
- net /Driver_U2_Out_B: track 0.00 -> 8.19 mm, vias 0 -> 2
- net D9~: track 61.5 -> 68.6 mm, vias 2 -> 3
- net Net-(Q2-G): track 12.2 -> 7.20 mm
- net ADS_ALERT: track 7.57 -> 12.4 mm, vias 2 -> 3
- net D7: track 47.4 -> 51.8 mm
- net GND: track 59.0 -> 55.2 mm, vias 12 -> 14
- net Net-(Q4-B): track 3.00 -> 0.00 mm
- net /V Signal to ADS: track 22.4 -> 24.8 mm
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
Commit message: Minor PCB Updates
Parts:
- moved RN2 30.5 mm to (118.8, 76.8)
- moved Q8 11.8 mm to (150.8, 78.9)
- moved R24 11.8 mm to (150.8, 82.3)
- moved Q7 5.12 mm to (123.2, 77.9)
- moved D4 5.11 mm to (136.2, 77.7)
- moved Q6 4.97 mm to (114.1, 77.7)
Connections:
- J1 pad 3: SDA -> +3V3
- J2 pad 6: SDA -> +3V3
- J6 pad 4: SDA -> +3V3
- Q6 pad 1: SDA -> +3V3
- Q7 pad 1: SDA -> +3V3
- RN2 pad 3: SDA -> +3V3
- RN2 pad 5: SDA -> +3V3
Routing:
- net +3V3: track 0.00 -> 69.5 mm, vias 0 -> 3
- net SDA: track 137.1 -> 79.5 mm, vias 7 -> 5
- net SCL-5V: track 35.5 -> 45.9 mm, vias 2 -> 3
- net VDD: track 158.0 -> 149.1 mm, vias 9 -> 10
- net /V Signal to ADS: track 24.8 -> 23.6 mm
- net SDA-5V: track 39.9 -> 39.0 mm

Commit message: PCB work
Parts:
- removed C6: ? DNP, Capacitor_SMD:C_0805_2012Metric_Pad1.18x1.45mm_HandSolder
- removed J4: IR Connection, Library:PinHeader_1x03_P2.54mm_Vertical_NoBox
- moved Q8 20.8 mm to (130.6, 84.2), turned to 90 degrees
- moved R24 20.0 mm to (131.5, 87.6), turned to 180 degrees
- moved JP6 7.07 mm to (122.5, 81.0), turned to 0 degrees
- moved D5 5.04 mm to (136.2, 83.2), turned to -90 degrees
Connections:
- net /V Ref to ADS renamed /V Ref to ADS-0
- net /V Signal to ADS renamed /ADC-1
Routing:
- net /Driver_U4_Out_A: track 0.00 -> 25.0 mm, vias 0 -> 2
- net GND: track 55.2 -> 64.9 mm
- net D5~ (IR): track 77.0 -> 67.7 mm, vias 2 -> 4
- net ADS_ADDR: track 4.62 -> 11.4 mm
- net /V Ref to ADS-0: track 23.5 -> 24.9 mm
- net VDD: track 149.1 -> 148.1 mm, vias 10 -> 9
Other:
- board text removed: "D5"
- board text removed: "IR"

Commit message: Finishing the next PCB version
Parts:
- added R7: 0, Resistor_SMD:R_0805_2012Metric_Pad1.20x1.40mm_HandSolder, F.Cu at (136.5, 60.8)
- added U5: Opamp_Dual, Package_SO:SOIC-8_3.9x4.9mm_P1.27mm, F.Cu at (134.3, 56.3)
- added U8: Opamp_Dual, Package_SO:SOIC-8_3.9x4.9mm_P1.27mm, F.Cu at (110.6, 59.0)
- moved Q1 2.85 mm to (90.2, 54.2)
- moved R1 2.13 mm to (91.6, 58.0)
Connections:
- J11 pad 2: I_Input -> Net-(J11-Pin_2)
- RN1 pad 2: SCL-5V -> SDA-5V
- RN1 pad 3: SDA-5V -> SCL-5V
Routing:
- net Net-(J11-Pin_2): track 0.00 -> 8.22 mm
- net I_Input: track 19.4 -> 11.4 mm
- net /V Ref to ADS-0: track 24.9 -> 31.0 mm
- net Net-(D1-A): track 5.35 -> 2.04 mm
- net ADS_ALERT: track 12.4 -> 9.81 mm
- net +9V: track 53.5 -> 51.3 mm
- net /ADC-1: track 23.2 -> 21.3 mm
- net Net-(Q1-B): track 3.33 -> 4.71 mm
- net A1/D15: track 80.7 -> 79.4 mm, vias 2 -> 1
- net VDD: track 148.1 -> 149.1 mm
- net GND: track 64.9 -> 64.1 mm
- net /R Circuit I Output: track 23.3 -> 22.8 mm
- net SDA: track 79.5 -> 79.7 mm, vias 5 -> 4
Other:
- outline, holes or cut-outs redrawn
