File: DMM_KiCAD_V4_next/DMM_KiCAD_V4_next.kicad_sch (KiCad schematic)
At the start: 81 parts, among them J1 Conn_01x07_Pin, J10 ANALOG, J11 I_Input, J12 Conn_01x02_Pin, J13 DIGITAL1, J14 Barrel_Jack, J15 Barrel_Jack, J16 Conn_01x01_Socket, J17 Conn_01x01_Socket, J2 MicoSD, J3 Conn_01x07_Pin, J5 POWER2, J6 POWER1, J7 Conn_01x02_Pin, J8 DIGITAL2, J9 Out to Screen, Q1 MMBT3904, Q2 AO3400A MOSFET, Q6 BSS138, Q7 BSS138, Q8 AO3400A MOSFET, SW1 SW_Push, SW2 SW_Push, SW3 SW_SPDT, SW4 SW_Push, U1 LM317_TO-220, U10 LM4040DBZ-2.5, U11 LM4040DBZ-5, U12 TLV61046ADBVR, U2 IX4426N, U3 ADS1115IDGS, U4 IX4426N, U5 Opamp_Dual, U7 MAX1683, U8 Opamp_Dual, U9 TPS613222ADBV

Commit message: New AdaLogger Version and PCB revisions
Parts:
- removed J1, J3: Conn_01x07_Pin, Connector_PinSocket_2.54mm:PinSocket_1x07_P2.54mm_Vertical, symbol Connector:Conn_01x07_Pin
- removed J10: ANALOG, Library:PinHeader_1x06_P2.54mm_Vertical_NoBox, symbol Connector_Generic:Conn_01x06
- removed J13: DIGITAL1, Library:PinHeader_1x08_P2.54mm_Vertical_NoBox, symbol Connector_Generic:Conn_01x08
- removed J5: POWER2, Library:PinHeader_1x03_P2.54mm_Vertical_NoBox, symbol Connector_Generic:Conn_01x03
- removed J6: POWER1, Library:PinHeader_1x08_P2.54mm_Vertical_NoBox, symbol Connector_Generic:Conn_01x08
- removed J8: DIGITAL2, Library:PinHeader_1x10_P2.54mm_Vertical_NoBox, symbol Connector_Generic:Conn_01x10
- removed JP6: Jumper_2_Bridged, Jumper:SolderJumper-2_P1.3mm_Bridged_Pad1.0x1.5mm, symbol Jumper:Jumper_2_Bridged
- removed Q6, Q7: BSS138, Package_TO_SOT_SMD:SOT-23, symbol Transistor_FET:BSS138
- removed R22: 0, Resistor_SMD:R_0805_2012Metric_Pad1.20x1.40mm_HandSolder, symbol Device:R_US
- removed RN2: 10k x4, Library:RESCAXS127P508X320X70-8N, symbol Device:R_Pack04_SIP
- removed U5, U8: Opamp_Dual, Package_SO:SOIC-8_3.9x4.9mm_P1.27mm, symbol Device:Opamp_Dual
- removed U6: ~, symbol Seeed_libdb:Module/XIAO-HALF-HOLE
- added C7, C8: 0.1uF, Capacitor_SMD:C_0805_2012Metric_Pad1.18x1.45mm_HandSolder, symbol Device:C
- added R12: 0, Resistor_SMD:R_0805_2012Metric_Pad1.20x1.40mm_HandSolder, symbol Device:R_US
- added RN3, RN4, RN5: 10k x4, Library:RESCAXS127P508X320X70-8N, symbol Device:R_Pack04_SIP
- added U13: ISO1540, Package_SO:SOIC-8_3.9x4.9mm_P1.27mm, symbol Isolator:ISO1540
- added U14: RFM-0505S, Converter_DCDC:Converter_DCDC_TRACO_TEA1-xxxx_THT, symbol CustomAdded:RFM_0505
- added U5, U8: LTV-824, Package_SO:SOP-8_6.605x9.655mm_P2.54mm, symbol Isolator:LTV-824
Connections:
- net ADS_ADDR: now also R12.1
- net D5~ (IR): now also U8.1; no longer U4.2 (IN_A)
- net D7: now also U5.1; no longer U2.2 (IN_A)
- net D9~: now also U5.3; no longer U2.4 (IN_B)
- net Driver_U4_In_B: now also RN4.3 (R3.1), U8.5
- net GND: now also C8.2, RN4.5 (R2.2), RN4.8 (R1.2), RN5.5 (R2.2), RN5.8 (R1.2), U13.4 (GND1), U14.1 (VIN-); no longer C10.1, C17.1, C18.2, C3.2, C4.1, D5.2 (A), F1.2, J11.3 (Pin_3), R6.1, U10.2 (A), U10.3 (nc_(gnd)), U11.2 (A), U11.3 (nc_(gnd)), U2.3 (GND), U3.3 (GND), U4.3 (GND), U7.1 (Gnd)
- net SCL: now also RN3.1 (R1.1), U13.3 (SCL1)
- net SCL-5V: now also RN3.7 (R4.2), U13.6 (SCL2)
- net SDA: now also RN3.4 (R2.1), U13.2 (SDA1)
- net SDA-5V: now also RN3.6 (R3.2), U13.7 (SDA2)
- net VDD: now also C8.1, RN3.5 (R2.2), RN3.8 (R1.2), U13.1 (VCC1), U14.2 (VIN+); no longer C4.2, D4.1 (K), J11.1 (Pin_1), R27.1, RN1.5 (R2.2), RN1.6 (R3.2), RN1.7 (R4.2), U3.8 (VDD), U7.4 (In)
- new net: RN4.4 (R2.1), U8.4
- new net: RN5.1 (R1.1), U5.2
- new net: RN4.1 (R1.1), U8.2
- new net: RN5.4 (R2.1), U5.4
- new net 5V-iso: C4.2, C7.1, D4.1 (K), J11.1 (Pin_1), R27.1, RN1.5 (R2.2), RN1.6 (R3.2), RN1.7 (R4.2), RN3.2 (R4.1), RN3.3 (R3.1), U13.8 (VCC2), U14.4 (Vout+), U3.8 (VDD), U5.6, U5.8, U7.4 (In), U8.6, U8.8
- new net Driver_U2_In_A: RN5.2 (R4.1), U2.2 (IN_A), U5.7
- new net Driver_U2_In_B: RN5.3 (R3.1), U2.4 (IN_B), U5.5
- new net Driver_U4_In_A: RN4.2 (R4.1), U4.2 (IN_A), U8.7
- new net Gnd-iso: C10.1, C17.1, C18.2, C3.2, C4.1, C7.2, D5.2 (A), F1.2, J11.3 (Pin_3), R12.2, R6.1, RN4.6 (R3.2), RN4.7 (R4.2), RN5.6 (R3.2), RN5.7 (R4.2), U10.2 (A), U10.3 (nc_(gnd)), U11.2 (A), U11.3 (nc_(gnd)), U13.5 (GND2), U14.3 (Vout-), U2.3 (GND), U3.3 (GND), U4.3 (GND), U7.1 (Gnd)
Other:
- added sheet ArduinoUnoPins (UnoPins.kicad_sch)
- added sheet XIAOPins (XIAOPins.kicad_sch)
- note removed: "XIAO PIN Header"
- moved on the sheet: C1, C10, C15, C16, C19, C2, C5, C6, C9, J17, J7, L1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
