File: DMM_KiCAD_V4_next/DMM_KiCAD_V4_next.kicad_pcb (KiCad board)
At the start: 4 copper layers, 68.5 x 53.2 mm, 76 parts, among them J1 Conn_01x07_Pin, J10 ANALOG, J11 I_Input, J12 Conn_01x02_Pin, J13 DIGITAL1, J14 Barrel_Jack, J15 Barrel_Jack, J16 Conn_01x01_Socket, J17 Conn_01x01_Socket, J2 MicoSD, J3 Conn_01x07_Pin, J5 POWER2, J6 POWER1, J7 Conn_01x02_Pin, J8 DIGITAL2, J9 Out to Screen, Q1 MMBT3904, Q2 AO3400A MOSFET, Q6 BSS138, Q7 BSS138, Q8 AO3400A MOSFET, SW1 SW_Push, SW2 SW_Push, SW3 SW_SPDT, SW4 SW_Push, U1 LM317_TO-220, U10 LM4040DBZ-2.5, U11 LM4040DBZ-5, U12 TLV61046ADBVR, U2 IX4426N, U3 ADS1115IDGS, U4 IX4426N, U5 Opamp_Dual, U7 MAX1683, U8 Opamp_Dual, U9 TPS613222ADBV

Commit message: Working on the next PCBs
Parts:
- added J18: DIOs_Extended, Connector_PinHeader_2.54mm:PinHeader_1x08_P2.54mm_Vertical, F.Cu at (146.9, 50.8)
- added J18: DIOs_Extended, Connector_PinHeader_2.54mm:PinHeader_1x08_P2.54mm_Vertical, F.Cu at (161.0, 59.5)
- added J19: Conn_01x02_Pin, Connector_PinSocket_2.54mm:PinSocket_1x02_P2.54mm_Vertical, F.Cu at (149.4, 100.1)
- added J4: A_Extended, Connector_PinHeader_2.54mm:PinHeader_1x08_P2.54mm_Vertical, F.Cu at (156.7, 99.6)
- RN1, RN2: footprint Resistor_SMD:R_Array_Convex_4x1206 -> Library:RESCAXS127P508X320X70-8N
- moved U8 65.7 mm to (133.8, 56.8)
- moved U5 43.5 mm to (110.9, 58.6)

Commit message: Work on next PCB version
Parts:
- moved J18 50.5 mm to (142.6, 106.5)
- moved J19 5.13 mm to (144.4, 99.1)
- moved J4 4.73 mm to (152.0, 99.1)
Changed lines of the file:
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@@
 	(footprint "Connector_PinSocket_2.54mm:PinSocket_1x02_P2.54mm_Vertical"
 		(layer "F.Cu")
-		(at 149.4 100.1 90)
+		(at 144.377549 99.070425 90)
 		(descr "Through hole straight socket strip, 1x02, 2.54mm pitch, single row (from Kicad 4.0.7), script generated")
 		(tags "Through hole socket strip THT 1x02 2.54mm single row")
@@
 	(footprint "Connector_PinHeader_2.54mm:PinHeader_1x08_P2.54mm_Vertical"
 		(layer "F.Cu")
-		(at 156.7 99.6 90)
+		(at 152 99.1 90)
 		(descr "Through hole straight pin header, 1x08, 2.54mm pitch, single row")
 		(tags "Through hole pin header THT 1x08 2.54mm single row")
@@
 	(footprint "Connector_PinHeader_2.54mm:PinHeader_1x08_P2.54mm_Vertical"
 		(layer "F.Cu")
-		(at 161 59.5 90)
+		(at 142.58 106.5 90)
 		(descr "Through hole straight pin header, 1x08, 2.54mm pitch, single row")
 		(tags "Through hole pin header THT 1x08 2.54mm single row")
