File: AnalogFrontEnd/AnalogFrontEnd.kicad_pcb (KiCad board)
At the start: 4 copper layers, 84.2 x 66.2 mm, 50 parts, among them J1 Voltmeter, J14 Barrel_Jack, J15 Barrel_Jack, J17 Conn_01x01_Socket, J7 Conn_01x02_Pin, J9 Out to Screen, Q1 MMBT3904, Q2 AO3400A MOSFET, Q6 BSS138, Q7 BSS138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

Commit message: Voltmeter Front End Conditioning PCB
Parts:
- added R3: 1K, Resistor_SMD:R_0805_2012Metric_Pad1.20x1.40mm_HandSolder, F.Cu at (168.5, 105.8)
- added SW3: SW_Push, Button_Switch_SMD:SW_SPST_CK_RS282G05A3, F.Cu at (168.4, 112.3)
- J1: footprint Connector_PinSocket_2.54mm:PinSocket_1x05_P2.54mm_Vertical -> Connector_PinSocket_2.54mm:PinSocket_1x06_P2.54mm_Vertical
- moved C9 135.2 mm to (175.3, 116.7), turned to 0 degrees
- moved U7 130.2 mm to (175.2, 113.0), turned to -90 degrees
- moved C10 125.0 mm to (175.3, 109.1), turned to 180 degrees
- moved Q7 90.8 mm to (151.3, 69.6)
- moved RN2 90.8 mm to (146.8, 68.5)
- moved Q6 90.8 mm to (142.2, 69.4)
- moved C16 71.4 mm to (107.1, 85.4)
- moved C19 71.4 mm to (107.1, 82.6)
- moved J17 71.4 mm to (100.1, 92.2)
- moved J7 71.4 mm to (102.0, 74.4)
- moved L1 71.4 mm to (107.0, 91.5)
- moved U9 71.4 mm to (107.0, 88.4)
- moved C15 71.4 mm to (108.3, 94.1)
- moved R23 71.4 mm to (108.7, 101.1)
- moved R2 57.5 mm to (133.8, 62.2)
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Routing:
- net VDD: track 24.2 -> 45.2 mm, vias 3 -> 4
- net VmeterMOSFET: track 22.6 -> 38.1 mm, vias 0 -> 2
- net GND: track 9.33 -> 23.6 mm, vias 4 -> 5
- net /ADC-1: track 16.6 -> 30.9 mm, vias 0 -> 1
- net +9V: track 18.3 -> 27.8 mm
- net /V Ref to ADS-0: track 22.9 -> 26.2 mm
- net /Driver_U4_Out_A: track 4.08 -> 6.17 mm
Other:
- board size 84.2 x 66.2 mm -> 46 x 24.4 mm
- board text added: "5V"
- board text added: "9V"
- board text added: "Charge Pump"
- board text added: "Ctrl"
- board text added: "OIH Designs Voltmeter Breakout V1"
- board text added: "Safety"
- board text added: "Voltmeter"
- board text added: "Voltmeter Front End: Above Gnd w Open Lead Detect Populate Charge pump or supply ~9vdc. Not Both. Remove/ DNP MOSFET to Disable Open Lead Detect."
- board text removed: "Charge Pump VIN x2"
- board text removed: "Protection"
- board text removed: "Q8"
- board text removed: "VIN"
- board text removed: "Voltmeter (open lead detect)"
