File: AnalogFrontEnd/AnalogFrontEnd.kicad_sch (KiCad schematic)
At the start: 54 parts, among them J1 Voltmeter, J14 Barrel_Jack, J15 Barrel_Jack, J17 Conn_01x01_Socket, J7 Conn_01x02_Pin, J9 Out to Screen, Q1 MMBT3904, Q2 AO3400A MOSFET, Q6 BSS138, Q7 BSS138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

Commit message: Voltmeter Front End Conditioning PCB
Parts:
- added R3: 1K, Resistor_SMD:R_0805_2012Metric_Pad1.20x1.40mm_HandSolder, symbol Device:R_US
- added SW3: SW_Push, Button_Switch_SMD:SW_SPST_CK_RS282G05A3, symbol Switch:SW_Push
- J1: footprint Connector_PinSocket_2.54mm:PinSocket_1x05_P2.54mm_Vertical -> Connector_PinSocket_2.54mm:PinSocket_1x06_P2.54mm_Vertical
Connections:
- net GND: now also SW3.2
- net VDD: now also R3.1
- net VmeterMOSFET: now also R3.2, SW3.1
