File: VoltmeterFrontEnd/_autosave-VoltmeterFrontEnd.kicad_sch (KiCad schematic)
At the start: 23 parts, among them J1 Voltmeter, J15 Barrel_Jack, Q3 MMBT3904, Q8 AO3400A MOSFET, SW3 SW_Push, U10 LM4040DBZ-2.5, U7 MAX1683

Commit message: Learning QSpice
Parts:
- R12: value 75K -> 100K
- R3: value 1K -> 10K
- R8: value 4.7K -> 10K
Connections:
- net +9V: now also R8.2; no longer R8.1
- net MOSFET_Gate: now also R8.1; no longer R8.2
Other:
- moved on the sheet: C17, R8, U10
