File: PCBDesigns/DMM_KiCAD_V4_UnoSpecific/DMM_KiCAD_V4_UnoSpecific.kicad_pcb (KiCad board)
At the start: 4 copper layers, 68.5 x 53.2 mm, 59 parts, among them J1 POWER2, J10 I_Input, J11 Conn_01x02_Pin, J2 POWER1, J3 DIGITAL2, J4 Out to Screen, J5 ANALOG, J6 DIGITAL1, J7 Barrel_Jack, J8 Conn_01x01_Socket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

Commit message: Working on Uno Form specific DMM
Parts:
- added J12: Conn_01x02_Pin, Connector_PinSocket_2.54mm:PinSocket_1x02_P2.54mm_Vertical, F.Cu at (113.0, 92.7)
- added R18: 1K, Resistor_SMD:R_0805_2012Metric_Pad1.20x1.40mm_HandSolder, F.Cu at (83.2, 85.7)
- added R19: 1K, Resistor_SMD:R_0805_2012Metric_Pad1.20x1.40mm_HandSolder, F.Cu at (82.8, 95.9)
- added RV1: 06TR4FA103DPR, Potentiometer_SMD:Potentiometer_ACP_CA6-VSMD_Vertical, F.Cu at (86.4, 80.6)
- added RV2: R_Potentiometer_US, Potentiometer_SMD:Potentiometer_ACP_CA6-VSMD_Vertical, F.Cu at (86.4, 90.8)
Routing:
- net A2/D16: track 0.00 -> 53.2 mm
- net A1/D15: track 0.00 -> 47.3 mm
- net GND: track 30.6 -> 54.2 mm, vias 5 -> 7
- net +VSW: track 4.69 -> 19.6 mm, vias 0 -> 2
- net VDD: track 32.3 -> 36.7 mm, vias 5 -> 7
- net Net-(R19-Pad1): track 0.00 -> 3.02 mm
- net Net-(R18-Pad1): track 0.00 -> 2.99 mm
- net 5V-iso: track 98.1 -> 96.4 mm
- net I_Input: track 11.4 -> 11.9 mm
Other:
- board text added: "BATT"
- board text removed: "EXT BATT"

Commit message: Finished(?) an Uno footprint board, started on Feather specific
Parts:
- removed F1: Fuse, Fuse:Fuse_1206_3216Metric_Pad1.42x1.75mm_HandSolder
Connections:
- J7 pad 2: Net-(F1-Pad1) -> Gnd-iso
Routing:
- net Net-(F1-Pad1): track 21.4 -> 0.00 mm, vias 1 -> 0
- net /ADC-1: track 15.9 -> 21.3 mm
- net 5V-iso: track 96.4 -> 94.0 mm, vias 8 -> 7
- net Gnd-iso: track 46.5 -> 44.6 mm
- net SCL-5V: track 49.0 -> 49.5 mm
