File: PCBDesigns/IsolatedADSandVoltmeterPCB/IsolatedADSandVoltmeterPCB.kicad_sch (KiCad schematic)
At the start: 27 parts, among them J1 Screw_Terminal_01x04, J15 Barrel_Jack, J2 Screw_Terminal_01x06, J3 Conn_01x04_MountingPin, J4 Conn_01x04_MountingPin, J5 Conn_01x04_MountingPin, U13 ISO1540, U14 RFM-0505S, U3 ADS1115IDGS

Commit message: Made a new logger version that can now do current and voltage simultaneously.
Parts:
- C4, C7, C8: Cost (10+) (none) -> 0.016; DigiKey Link (none) -> https://www.digikey.com/en/products/detail/kemet/C0805C104K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
- D4, D5: Cost (10+) (none) -> 0.05; DigiKey Link (none) -> https://www.digikey.com/en/products/detail/onsemi/BAT54T1G/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
- J3, J4, J5: Cost (10+) (none) -> 0.42; DigiKey Link (none) -> https://www.digikey.com/en/products/detail/jst-sales-americ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
- R1, R2, R5, R6, R7: value 4.7K -> 1K; Cost (10+) (none) -> 0.03; DigiKey Link (none) -> https://www.digikey.com/en/products/detail/susumu/RR1220P-1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
- R12: value 0 -> 1K; Cost (10+) (none) -> 0.03; DigiKey Link (none) -> https://www.digikey.com/en/products/detail/susumu/RR1220P-1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
- R17, R18: Cost (10+) (none) -> 0.08; DigiKey Link (none) -> https://www.digikey.com/en/products/detail/susumu/RG2012P-4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
- R24: Cost (10+) (none) -> 0.06; DigiKey Link (none) -> https://www.digikey.com/en/products/detail/panasonic-electr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
- U13: Cost (10+) (none) -> 3.45; DigiKey Link (none) -> https://www.digikey.com/en/products/detail/texas-instrument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
- U14: Cost (10+) (none) -> 2.51; DigiKey Link (none) -> https://www.digikey.com/en/products/detail/xp-power/SCT01F0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
- U3: Cost (10+) (none) -> 2.23; DigiKey Link (none) -> https://www.digikey.com/en/products/detail/texas-instrument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
