File: PCBDesigns/AMC0330R_Mount/AMC0330R_Mount.kicad_pcb (KiCad board)
At the start: 2 copper layers, 45.7 x 24 mm, 13 parts, among them J1 HV_Input, J2 Low_Side, U1 AMC0330R-Q1, U2 RFM-0505S

Commit message: Added smoothing to generic voltmeter, and worked on AMC0330R PCB
Parts:
- moved J1 12.8 mm to (90.8, 74.3)
- moved J2 3.27 mm to (116.2, 74.3)
- moved C5 2.88 mm to (86.2, 76.2)
- moved C1 2.40 mm to (91.4, 81.9)
- moved R1 2.39 mm to (83.2, 71.8)
- moved C2 2.30 mm to (88.3, 81.9)
- moved R2 1.53 mm to (83.2, 76.2)
- moved R3 1.24 mm to (85.2, 81.0)
- moved C4 0.72 mm to (112.4, 79.6)
- moved C3 0.42 mm to (109.9, 79.6)
Routing:
- net GND1: track 43.2 -> 14.2 mm
- net GND2: track 35.1 -> 9.75 mm, vias 1 -> 2
- net OUT: track 14.6 -> 11.1 mm, vias 1 -> 0
- net 5V_IN: track 20.9 -> 17.4 mm
- net VDD1: track 22.9 -> 20.0 mm
- net Net-(J1-Pin_1): track 6.83 -> 9.62 mm
- net VDD2: track 19.6 -> 21.5 mm
- net Net-(R1-Pad2): track 1.50 -> 2.45 mm
Other:
- board size 45.7 x 24 mm -> 40 x 19.7 mm

Commit message: Various troubleshooting and PCB design
Parts:
- removed J1: HV_Input, Connector_PinHeader_2.54mm:PinHeader_1x02_P2.54mm_Vertical
- added J14: Barrel_Jack, Connector_BarrelJack:BarrelJack_Horizontal, F.Cu at (85.1, 76.8)
- moved C5 8.50 mm to (94.6, 77.5), turned to 0 degrees
- moved R2 7.73 mm to (90.8, 74.9)
- moved R1 5.72 mm to (88.9, 71.8), turned to 0 degrees
- moved R3 5.42 mm to (90.2, 78.7), turned to 180 degrees
- moved C3 4.68 mm to (109.9, 74.9)
- moved J2 2.62 mm to (113.7, 73.7)
- moved C4 2.54 mm to (109.9, 79.6)
- moved C2 1.91 mm to (90.2, 81.9)
- moved C1 1.84 mm to (93.3, 81.9)
- moved U1 1.60 mm to (101.6, 82.0)
- moved U2 1.06 mm to (104.1, 69.8)
- moved C6 0.14 mm to (109.9, 84.0)
Routing:
- net Net-(U1-INP): track 18.1 -> 11.5 mm
- net GND1: track 14.2 -> 9.25 mm, vias 2 -> 4
- net OUT: track 11.1 -> 6.76 mm
- net Net-(J14-Pad1): track 9.62 -> 6.88 mm
- net 5V_IN: track 17.4 -> 14.9 mm
- net VDD1: track 20.0 -> 17.6 mm
- net VDD2: track 21.5 -> 20.4 mm
Other:
- board size 40 x 19.7 mm -> 39.3 x 19.7 mm
- board text added: "5V IN"
- board text added: "AMC0330R Dev Board"
- board text added: "Gnd"
- board text added: "HIGH"
- board text added: "LOW"
- board text added: "Signal Out"
- board text added: "VIN+"
- board text added: "VIN-"
- board text added: "Vdd"
- board text removed: "HIGH SIDE"
- board text removed: "LOW SIDE"
