File: PCBDesigns/AMC0330R_Mount/AMC0330R_Mount.kicad_sch (KiCad schematic)
At the start: 13 parts, among them J1 HV_Input, J2 Low_Side, U1 AMC0330R-Q1, U2 RFM-0505S

Commit message: Added smoothing to generic voltmeter, and worked on AMC0330R PCB
Other:
- moved on the sheet: C5
Changed lines of the file:
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@@
+	)
+	(junction
+		(at 78.74 73.66)
+		(diameter 0)
+		(color 0 0 0 0)
 	)
 	(junction
@@
 	(wire
 		(pts
+			(xy 127 91.44) (xy 125.73 91.44)
+		)
+		(stroke
+			(width 0)
+			(type default)
+		)
+	)
+	(wire
+		(pts
 			(xy 30.48 78.74) (xy 35.56 78.74)
 		)
@@
 	(wire
 		(pts
-			(xy 78.74 77.47) (xy 78.74 80.01)
+			(xy 78.74 77.47) (xy 78.74 78.74)
 		)
 		(stroke
@@
 	(wire
 		(pts
+			(xy 91.44 73.66) (xy 91.44 74.93)
+		)
+		(stroke
+			(width 0)
+			(type default)
+		)
+	)
+	(wire
+		(pts
+			(xy 111.76 74.93) (xy 116.84 74.93)
+		)
+		(stroke
+			(width 0)
+			(type default)
+		)
+	)
+	(wire
+		(pts
+			(xy 83.82 59.69) (xy 88.9 59.69)
+		)
+		(stroke
+			(width 0)
+			(type default)
+		)
+	)
+	(wire
+		(pts
+			(xy 85.09 80.01) (xy 85.09 77.47)
+		)
+		(stroke
+			(width 0)
+			(type default)
+		)
+	)
+	(wire
+		(pts
+			(xy 30.48 76.2) (xy 30.48 54.61)
+		)
+		(stroke
+			(width 0)
+			(type default)
+		)
+	)
+	(wire
+		(pts
+			(xy 111.76 72.39) (xy 111.76 67.31)
+		)
+		(stroke
+			(width 0)
+			(type default)
+		)
+	)
+	(wire
+		(pts
 			(xy 45.72 62.23) (xy 45.72 66.04)
 		)
@@
 	(wire
 		(pts
-			(xy 91.44 73.66) (xy 91.44 74.93)
-		)
-		(stroke
-			(width 0)
-			(type default)
-		)
-	)
-	(wire
-		(pts
-			(xy 111.76 74.93) (xy 116.84 74.93)
-		)
-		(stroke
-			(width 0)
-			(type default)
-		)
-	)
-	(wire
-		(pts
-			(xy 83.82 59.69) (xy 88.9 59.69)
-		)
-		(stroke
-			(width 0)
-			(type default)
-		)
-	)
-	(wire
-		(pts
-			(xy 85.09 80.01) (xy 85.09 77.47)
-		)
-		(stroke
-			(width 0)
-			(type default)
-		)
-	)
-	(wire
-		(pts
-			(xy 30.48 76.2) (xy 30.48 54.61)
-		)
-		(stroke
-			(width 0)
-			(type default)
-		)
-	)
-	(wire
-		(pts
-			(xy 111.76 72.39) (xy 111.76 67.31)
-		)
-		(stroke
-			(width 0)
-			(type default)
-		)
-	)
-	(wire
-		(pts
 			(xy 116.84 59.69) (xy 128.27 59.69)
 		)
@@
 	(wire
 		(pts
+			(xy 127 83.82) (xy 125.73 83.82)
+		)
+		(stroke
+			(width 0)
+			(type default)
+		)
+	)
+	(wire
+		(pts
 			(xy 91.44 80.01) (xy 85.09 80.01)
 		)
@@
 	(wire
 		(pts
-			(xy 78.74 73.66) (xy 78.74 72.39)
+			(xy 78.74 73.66) (xy 78.74 71.12)
 		)
 		(stroke
@@
 	(global_label "VDD2"
 		(shape bidirectional)
-		(at 125.73 83.82 0)
-		(effects
-			(font
-				(size 1.27 1.27)
-			)
-			(justify left)
-		)
-		(property "Intersheetrefs" "${INTERSHEET_REFS}"
-			(at 135.73 83.82 0)
+		(at 127 83.82 0)
+		(effects
+			(font
+				(size 1.27 1.27)
+			)
+			(justify left)
+		)
+		(property "Intersheetrefs" "${INTERSHEET_REFS}"
+			(at 137 83.82 0)
 			(effects
 				(font
@@
 	(global_label "GND2"
 		(shape bidirectional)
-		(at 125.73 91.44 0)
-		(effects
-			(font
-				(size 1.27 1.27)
-			)
-			(justify left)
-		)
-		(property "Intersheetrefs" "${INTERSHEET_REFS}"
-			(at 135.73 91.44 0)
+		(at 127 91.44 0)
+		(effects
+			(font
+				(size 1.27 1.27)
+			)
+			(justify left)
+		)
+		(property "Intersheetrefs" "${INTERSHEET_REFS}"
+			(at 137 91.44 0)
 			(effects
 				(font
@@
 	(symbol
 		(lib_id "Device:C")
-		(at 78.74 76.2 0)
+		(at 78.74 74.93 0)
 		(unit 1)
 		(exclude_from_sim no)
@@
 		(dnp no)
 		(property "Reference" "C5"
-			(at 78.74 71.12 0)
+			(at 78.74 69.85 0)
 			(effects
 				(font
@@
 		)
 		(property "Value" "100pF"
-			(at 78.74 81.28 0)
+			(at 78.74 80.01 0)
 			(effects
 				(font
@@
 		)
 		(property "Footprint" "Capacitor_SMD:C_0805_2012Metric_Pad1.18x1.45mm_HandSolder"
-			(at 78.74 76.2 0)
+			(at 78.74 74.93 0)
 			(effects
 				(font
@@
 		)
 		(property "Datasheet" "~"
-			(at 78.74 76.2 0)
+			(at 78.74 74.93 0)
 			(effects
 				(font
@@
 		)
 		(property "Description" "Unpolarized capacitor"
-			(at 78.74 76.2 0)
-			(effects
-				(font
+			(at 78.74 74.93 0)
+			(effects
+				(font

Commit message: Various troubleshooting and PCB design
Parts:
- removed J1: HV_Input, Connector_PinHeader_2.54mm:PinHeader_1x02_P2.54mm_Vertical, symbol Connector_Generic:Conn_01x02
- added J14: Barrel_Jack, Connector_BarrelJack:BarrelJack_Horizontal, symbol Connector:Barrel_Jack
- U2: value RFM-0505S -> SCT01F03S05
Connections:
- net GND1: now also J14.2
- net at R1.1: now also J14.1
Other:
- moved on the sheet: J2, R1, R2, R3
