File: PCBDesigns/DualAMCBoard/DualAMCBoard.kicad_sch (KiCad schematic)
At the start: 59 parts, among them J1 Screw_Terminal_01x02, J11 Differential Out, J6 Screw_Terminal_01x02, J7 Power Input, J8 Differential Out, J9 SE Out, U1 OPA2191ID

Commit message: Work on different PCBs. Mostly.
Changed lines of the file:
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@@
 	)
 	(junction
-		(at 213.36 130.81)
+		(at 208.28 116.84)
 		(diameter 0)
 		(color 0 0 0 0)
 	)
 	(junction
-		(at 208.28 116.84)
+		(at 237.49 73.66)
 		(diameter 0)
 		(color 0 0 0 0)
 	)
 	(junction
-		(at 237.49 73.66)
+		(at 219.71 48.26)
 		(diameter 0)
 		(color 0 0 0 0)
@@
 	)
 	(junction
-		(at 219.71 48.26)
-		(diameter 0)
-		(color 0 0 0 0)
-	)
-	(junction
 		(at 58.42 139.7)
 		(diameter 0)
@@
 	)
 	(junction
-		(at 236.22 149.86)
-		(diameter 0)
-		(color 0 0 0 0)
-	)
-	(junction
 		(at 104.14 118.11)
 		(diameter 0)
@@
 	)
 	(junction
-		(at 212.09 140.97)
-		(diameter 0)
-		(color 0 0 0 0)
-	)
-	(junction
 		(at 194.31 64.77)
 		(diameter 0)
@@
 	)
 	(junction
-		(at 219.71 64.77)
+		(at 237.49 57.15)
 		(diameter 0)
 		(color 0 0 0 0)
 	)
 	(junction
-		(at 237.49 57.15)
+		(at 220.98 124.46)
 		(diameter 0)
 		(color 0 0 0 0)
@@
 	)
 	(junction
-		(at 220.98 124.46)
-		(diameter 0)
-		(color 0 0 0 0)
-	)
-	(junction
 		(at 113.03 115.57)
 		(diameter 0)
@@
 	(wire
 		(pts
-			(xy 220.98 121.92) (xy 220.98 124.46)
-		)
-		(stroke
-			(width 0)
-			(type default)
-		)
-	)
-	(wire
-		(pts
 			(xy 152.4 39.37) (xy 154.94 39.37)
 		)
@@
 	(wire
 		(pts
-			(xy 236.22 149.86) (xy 233.68 149.86)
-		)
-		(stroke
-			(width 0)
-			(type default)
-		)
-	)
-	(wire
-		(pts
 			(xy 194.31 64.77) (xy 212.09 64.77)
 		)
@@
 	(wire
 		(pts
-			(xy 215.9 45.72) (xy 219.71 45.72)
+			(xy 215.9 48.26) (xy 219.71 48.26)
 		)
 		(stroke
@@
 	(wire
 		(pts
+			(xy 217.17 124.46) (xy 217.17 121.92)
+		)
+		(stroke
+			(width 0)
+			(type default)
+		)
+	)
+	(wire
+		(pts
 			(xy 60.96 60.96) (xy 60.96 63.5)
 		)
@@
 	(wire
 		(pts
-			(xy 87.63 62.23) (xy 87.63 63.5)
+			(xy 215.9 48.26) (xy 215.9 45.72)
 		)
 		(stroke
@@
 	(wire
 		(pts
-			(xy 58.42 147.32) (xy 58.42 139.7)
+			(xy 87.63 62.23) (xy 87.63 63.5)
 		)
 		(stroke
@@
 	(wire
 		(pts
-			(xy 213.36 130.81) (xy 214.63 130.81)
+			(xy 58.42 147.32) (xy 58.42 139.7)
 		)
 		(stroke
@@
 	(wire
 		(pts
-			(xy 219.71 130.81) (xy 220.98 130.81)
-		)
-		(stroke
-			(width 0)
-			(type default)
-		)
-	)
-	(wire
-		(pts
 			(xy 66.04 129.54) (xy 62.23 129.54)
 		)
@@
 	(wire
 		(pts
-			(xy 219.71 45.72) (xy 219.71 48.26)
-		)
-		(stroke
-			(width 0)
-			(type default)
-		)
-	)
-	(wire
-		(pts
 			(xy 88.9 129.54) (xy 88.9 133.35)
 		)
@@
 	(wire
 		(pts
-			(xy 218.44 64.77) (xy 219.71 64.77)
-		)
-		(stroke
-			(width 0)
-			(type default)
-		)
-	)
-	(wire
-		(pts
 			(xy 110.49 58.42) (xy 90.17 58.42)
 		)
@@
 	(wire
 		(pts
-			(xy 217.17 121.92) (xy 220.98 121.92)
+			(xy 217.17 124.46) (xy 220.98 124.46)
 		)
 		(stroke
@@
 	(wire
 		(pts
-			(xy 212.09 140.97) (xy 214.63 140.97)
-		)
-		(stroke
-			(width 0)
-			(type default)
-		)
-	)
-	(wire
-		(pts
 			(xy 102.87 55.88) (xy 102.87 62.23)
 		)
@@
 		(in_pos_files yes)
 		(dnp no)
-		(fields_autoplaced yes)
 		(property "Reference" "RN3"
-			(at 222.25 43.1799 0)
+			(at 222.25 39.878 0)
 			(show_name no)
 			(do_not_autoplace no)
@@
 		)
 		(property "Value" "R_Pack04_Split"
-			(at 222.25 45.7199 0)
+			(at 222.25 42.418 0)
 			(show_name no)
 			(do_not_autoplace no)
@@
 		(in_pos_files yes)
 		(dnp no)
-		(fields_autoplaced yes)
 		(property "Reference" "RN4"
-			(at 217.17 124.46 90)
+			(at 214.376 125.222 90)
 			(show_name no)
 			(do_not_autoplace no)
@@
 		(in_pos_files yes)
 		(dnp no)
-		(fields_autoplaced yes)
 		(property "Reference" "RN3"
-			(at 214.63 48.26 90)
+			(at 212.09 49.276 90)
 			(show_name no)
 			(do_not_autoplace no)
