File: PCBDesigns/DMM Giga Shield Version/DMM Giga Shield Version.kicad_sch (KiCad schematic)
At the start: 82 parts, among them J1 TRRS, J10 ANALOG, J11 I_Input, J12 Conn_01x02_Pin, J13 DIGITAL1, J14 Barrel_Jack, J15 Barrel_Jack, J16 Conn_01x01_Socket, J17 Conn_01x01_Socket, J18 DIOs_Extended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

Commit message: PCB Work.
Other:
- moved on the sheet: C10, C9, U7
