File: PCBDesigns/FeatherVoltmeterPCBA/FeatherVoltmeterPCBA.kicad_pcb (KiCad board)
At the start: 4 copper layers, 23.5 x 51.1 mm, 35 parts, among them J1 Conn_01x16_Pin, J2 Conn_01x12_Pin, J5 Screw_Terminal_01x02, Q8 AO3400A MOSFET, SW1 SSSS811101, U1 ADuM1200AR, U10 LM4040DBZ-2.5, U13 ISO1540, U3 ADS1015

Commit message: PCB Work.
Other:
- board text added: "Address Alt"
Changed lines of the file:
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@@
 		(layer "Edge.Cuts")
 	)
-	(gr_text "SDA"
-		(at 130.683 85.598 0)
+	(gr_text "5V"
+		(at 130.683 84.074 0)
 		(layer "B.SilkS")
 		(effects
@@
 		)
 	)
-	(gr_text "SCL"
-		(at 130.683 88.519 0)
+	(gr_text "SDA"
+		(at 130.683 86.487 0)
 		(layer "B.SilkS")
 		(effects
@@
 		)
 	)
-	(gr_text "5V"
-		(at 133.985 81.661 0)
+	(gr_text "SCL"
+		(at 130.683 89.154 0)
 		(layer "B.SilkS")
 		(effects
@@
 	(gr_text "GND"
 		(at 134.112 91.186 0)
+		(layer "B.SilkS")
+		(effects
+			(font
+				(size 0.762 0.762)
+			)
+			(justify left bottom mirror)
+		)
+	)
+	(gr_text "Address Alt"
+		(at 128.143 83.058 90)
 		(layer "B.SilkS")
 		(effects
@@
 	)
 	(segment
-		(start 127.443 91.313)
-		(end 128.417999 91.313)
-		(width 0.2)
-		(layer "F.Cu")
-		(net "SDA-5V")
-	)
-	(segment
 		(start 131.445 96.863)
 		(end 131.426 96.882)
@@
 	)
 	(segment
-		(start 130.302 89.428999)
-		(end 130.302 86.36)
-		(width 0.2)
-		(layer "F.Cu")
-		(net "SDA-5V")
-	)
-	(segment
 		(start 131.445 96.710502)
 		(end 131.445 96.863)
@@
 	)
 	(segment
+		(start 130.302 89.428999)
+		(end 128.417999 91.313)
+		(width 0.2)
+		(layer "F.Cu")
+		(net "SDA-5V")
+	)
+	(segment
 		(start 131.426 97.787652)
 		(end 132.150201 98.511853)
@@
 	(segment
 		(start 128.417999 91.313)
+		(end 127.443 91.313)
+		(width 0.2)
+		(layer "F.Cu")
+		(net "SDA-5V")
+	)
+	(segment
+		(start 130.302 87.503)
 		(end 130.302 89.428999)
 		(width 0.2)
@@
 	)
 	(via
-		(at 130.302 86.36)
+		(at 130.302 87.503)
 		(size 0.6)
 		(drill 0.3)
@@
 	(segment
 		(start 130.683 85.979)
-		(end 130.302 86.36)
+		(end 131.609 85.979)
 		(width 0.2)
 		(layer "B.Cu")
@@
 	)
 	(segment
-		(start 131.609 85.979)
-		(end 130.683 85.979)
+		(start 130.302 87.503)
+		(end 130.302 86.36)
 		(width 0.2)
 		(layer "B.Cu")
@@
 		(width 0.2)
 		(layer "B.Cu")
+		(net "SDA-5V")
+	)
+	(segment
+		(start 130.302 86.36)
+		(end 130.683 85.979)
+		(width 0.2)
+		(layer "B.Cu")
