File: PCBDesigns/DMM Feather Redux/DMM Feather Redux.kicad_sch (KiCad schematic)
At the start: 50 parts, among them J10 I_Input, J14 Barrel_Jack, J2 Conn_01x03_Pin, J3 Conn_01x04_MountingPin, J7 Barrel_Jack, Q2 AO3400A MOSFET, Q8 AO3400A MOSFET, SW3 SW_SPDT, U1 ISO1644DWR, U10 LM4040DBZ-2.5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

Commit message: Work on different PCBs. Mostly.
Parts:
- removed A1: Adafruit_Feather_32u4_BluefruitLE, Module:Adafruit_Feather_WithMountingHoles, symbol MCU_Module:Adafruit_Feather_32u4_BluefruitLE
- removed J2: Conn_01x03_Pin, Connector_PinHeader_2.54mm:PinHeader_1x03_P2.54mm_Vertical, symbol Connector:Conn_01x03_Pin
- removed R6, R7: 4.7K, Resistor_SMD:R_0805_2012Metric_Pad1.20x1.40mm_HandSolder, symbol Device:R_US
- removed U1: ISO1644DWR, Package_SO:SOIC-16W_7.5x10.3mm_P1.27mm, symbol Isolator:ISO1644DWR
- added A2: Adafruit_Feather_32u4_BluefruitLE, Module:Adafruit_Feather_WithMountingHoles, symbol MCU_Module:Adafruit_Feather_32u4_BluefruitLE
- added D1: LED, LED_SMD:LED_Luminus_MP-3030-1100_3.0x3.0mm, symbol Device:LED
- added J5: Conn_01x12_Pin, Connector_PinSocket_2.54mm:PinSocket_1x12_P2.54mm_Vertical, symbol Connector:Conn_01x12_Pin
- added J6: Conn_01x16_Pin, Connector_PinSocket_2.54mm:PinSocket_1x16_P2.54mm_Vertical, symbol Connector:Conn_01x16_Pin
- added J9: Out to Screen, Connector_PinSocket_2.54mm:PinSocket_1x04_P2.54mm_Vertical, symbol Connector:Conn_01x04_Pin
- added Q1: MMBT3904, Package_TO_SOT_SMD:SOT-23, symbol Transistor_BJT:MMBT3904
- added R4: 500, Resistor_SMD:R_0805_2012Metric_Pad1.20x1.40mm_HandSolder, symbol Device:R_US
- added RN1: R_Pack04_Split, Resistor_SMD:R_Array_Convex_4x0603, symbol Device:R_Pack04_Split
- added SW1, SW2, SW4: SW_Push, Button_Switch_SMD:SW_SPST_CK_RS282G05A3, symbol Switch:SW_Push
- C17, C4, C7, C8: footprint Capacitor_SMD:C_0805_2012Metric_Pad1.18x1.45mm_HandSolder -> Capacitor_SMD:C_0603_1608Metric
- R1, R10, R11, R12, R19, R2, R27: footprint Resistor_SMD:R_0805_2012Metric_Pad1.20x1.40mm_HandSolder -> Resistor_SMD:R_0603_1608Metric
- R5: value 4.7K -> 1K; footprint Resistor_SMD:R_0805_2012Metric_Pad1.20x1.40mm_HandSolder -> Resistor_SMD:R_0603_1608Metric; Function (none) -> I limit for Q1
Connections:
- net Driver_U2_Out_B is gone; now on net I_Supply_Ohmmeter: U5.3 (VI)
- net 5V-iso: now also R4.2, RN1.1 (R1.1), RN1.3 (R3.1), RN1.4 (R4.1); no longer R5.1
- net ADS_ALERT: now also RN1.8 (R1.2)
- net D10_(Ohmmeter_I_ctrl): now also A2.22 (D10), J5.7 (Pin_7)
- net D9_(OhmmeterBridge_ctrl): now also A2.21 (D9), J5.8 (Pin_8)
- net GND: now also A2.4 (GND), J6.4 (Pin_4), J9.4 (Pin_4), SW1.2, SW2.2, SW4.2
- net Gnd-iso: now also D1.1 (K)
- net SCL: now also A2.18 (SCL/D3), J5.11 (Pin_11)
- net SCL-5V: now also J9.2 (Pin_2), RN1.5 (R4.2); no longer R5.2
- net SDA: now also A2.17 (SDA/D2), J5.12 (Pin_12)
- net SDA-5V: now also J9.1 (Pin_1), RN1.6 (R3.2)
- net VDD: now also A2.2 (3V3), J6.2 (Pin_2), J9.3 (Pin_3)
- net V_Bridge_Ctrl-MCU: now also A2.19 (D5), J5.10 (Pin_10)
- net LED_Ctrl_ISO: now reaches U4.11 (VOD)
- net LED_Ctrl_ISO: now also R5.1
- net LED_Ctrl: now reaches U4.6 (VID)
- net LED_Ctrl: now also A2.20 (D6)
- net at SW3.2 (B): now also A2.27 (EN), J5.2 (Pin_2)
- net MOSFET_Gate renamed V_Bridge_Ctrl-ISO
- new net: Q1.3 (C), R4.1
- new net: Q1.1 (B), R5.2
- new net: D1.2 (A), Q1.2 (E)
- new net D11: A2.23 (D11), SW4.1
- new net D12: A2.24 (D12), SW2.1
- new net D13: A2.25 (D13), SW1.1
Other:
- moved on the sheet: SW3

Commit message: More PCB work.
Parts:
- removed H1, H2, H3: MountingHole, MountingHole:MountingHole_2.2mm_M2_Pad, symbol Mechanical:MountingHole
- removed H4: MountingHole, MountingHole:MountingHole_2.2mm_M2_ISO14580, symbol Mechanical:MountingHole
Connections:
- net 5V-iso: now also RN1.2 (R2.1)
- net D11: now also J5.6 (Pin_6)
- net D12: now also J5.5 (Pin_5)
- net D13: now also J5.4 (Pin_4)
- net SCL: now also J9.2 (Pin_2)
- net SCL-5V: no longer J9.2 (Pin_2)
- net SDA: now also J9.1 (Pin_1)
- net SDA-5V: no longer J9.1 (Pin_1)
- net VDD: now also J6.3 (Pin_3)
- net RESET: now reaches J6.1 (Pin_1)
- net A5: now reaches J6.10 (Pin_10)
- net A5: now also A2.10 (A5)
- net SCK: now reaches J6.11 (Pin_11)
- net SCK: now also A2.11 (SCK/D15)
- net MOSI: now reaches J6.12 (Pin_12)
- net MOSI: now also A2.12 (MOSI/D16)
- net MISO: now reaches J6.13 (Pin_13)
- net MISO: now also A2.13 (MISO/D14)
- net RX: now reaches J6.14 (Pin_14)
- net RX: now also A2.14 (RX/D0)
- net TX: now reaches J6.15 (Pin_15)
- net TX: now also A2.15 (TX/D1)
- net A0: now reaches J6.5 (Pin_5)
- net A0: now also A2.5 (A0)
- net A1: now reaches J6.6 (Pin_6)
- net A1: now also A2.6 (A1)
- net A2: now reaches J6.7 (Pin_7)
- net A2: now also A2.7 (A2)
- net A3: now reaches J6.8 (Pin_8)
- net A3: now also A2.8 (A3)
- net A4: now reaches J6.9 (Pin_9)
- net A4: now also A2.9 (A4)
- net USB: now reaches A2.26 (USB)
- net USB: now also J5.3 (Pin_3)
- net EN: now reaches A2.27 (EN), J5.2 (Pin_2), SW3.2 (B)
- net VBAT: now reaches A2.28 (VBAT)
- net VBAT: now also J5.1 (Pin_1)
- net D6: now reaches J5.9 (Pin_9)
- net D6: now also A2.20 (D6), U4.4 (VIB)
- net D10_(Ohmmeter_I_ctrl) renamed D10
- net D10: now also U4.6 (VID); no longer U4.4 (VIB)
- net D9_(OhmmeterBridge_ctrl) renamed D9
- net D9: now also U4.5 (VIC); no longer U4.3 (VIA)
- removed net LED_Ctrl: A2.20 (D6), U4.6 (VID)
- net V_Bridge_Ctrl-MCU renamed D5
- net D5: now also U4.3 (VIA); no longer U4.5 (VIC)
Other:
- moved on the sheet: A2, J5, J6, J9, SW1, SW2, SW3, SW4

Commit message: PCB Work.
Parts:
- removed SW3: SW_SPDT, Button_Switch_THT:SW_Slide_SPDT_Angled_CK_OS102011MA1Q, symbol Switch:SW_SPDT
- added C10, C11: 0.1uF, Capacitor_SMD:C_0603_1608Metric, symbol Device:C
- added SW5: MS-22D28-G020, easyeda_parts:SW-SMD_MS-22D28-G020, symbol CustomAdded:MS-22D28-G020
- J3: now not fitted
Connections:
- net 5V-iso: now also C11.1
- net EN: now also SW5.3
- net GND: now also C10.2, SW5.2
- net Gnd-iso: now also C11.2
- net VDD: now also C10.1

Commit message: PCB Work
Parts:
- SW1, SW2, SW4: footprint Button_Switch_SMD:SW_SPST_CK_RS282G05A3 -> Button_Switch_SMD:SW_Push_1P1T-SH_NO_CK_KMR2xxG
Changed lines of the file:
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@@
 			)
 		)
-		(property "Footprint" "Button_Switch_SMD:SW_SPST_CK_RS282G05A3"
+		(property "Footprint" "Button_Switch_SMD:SW_Push_1P1T-SH_NO_CK_KMR2xxG"
 			(at 41.91 125.73 0)
 			(hide yes)
@@
 			)
 		)
-		(property "Footprint" "Button_Switch_SMD:SW_SPST_CK_RS282G05A3"
+		(property "Footprint" "Button_Switch_SMD:SW_Push_1P1T-SH_NO_CK_KMR2xxG"
 			(at 41.91 105.41 0)
 			(hide yes)
@@
 			)
 		)
-		(property "Footprint" "Button_Switch_SMD:SW_SPST_CK_RS282G05A3"
+		(property "Footprint" "Button_Switch_SMD:SW_Push_1P1T-SH_NO_CK_KMR2xxG"
 			(at 41.91 115.57 0)
 			(hide yes)

Commit message: DMM PCB work and Voltmeter Sketch Updates
Parts:
- removed SW5: MS-22D28-G020, easyeda_parts:SW-SMD_MS-22D28-G020, symbol CustomAdded:MS-22D28-G020
- added C12, C14: 10uF, Capacitor_SMD:C_0603_1608Metric, symbol Device:C
- added C13, C15: 0.1uF, Capacitor_SMD:C_0603_1608Metric, symbol Device:C
- added SW3: SW_SPDT, symbol Switch:SW_SPDT
- D1: footprint LED_SMD:LED_Luminus_MP-3030-1100_3.0x3.0mm -> Custom:LED-SMD_L3.0-W3.0_WHITE
- J5, J6: now fitted
Connections:
- net 5V-iso: now also C12.1, C13.1
- net D11: now also SW1.1; no longer SW4.1
- net D13: now also SW4.1; no longer SW1.1
- net EN: now also SW3.2 (B)
- net GND: now also C14.1, C15.1, SW3.3 (C)
- net Gnd-iso: now also D1.2 (K), C12.2, C13.2; no longer D1.1 (K)
- net VDD: now also C14.2, C15.2
- net at Q1.2 (E): now also D1.1 (A); no longer D1.2 (A)

Commit message: Circuits, mostly
Parts:
- removed SW3: SW_SPDT, symbol Switch:SW_SPDT
- added J1, J2: Conn_01x02, Connector_PinSocket_2.54mm:PinSocket_1x02_P2.54mm_Vertical, symbol Connector_Generic:Conn_01x02
- added R20, R21: 240k, Resistor_SMD:R_0805_2012Metric, symbol Device:R_US
- R14, R24, R3, R4, R8, R9: footprint Resistor_SMD:R_0805_2012Metric_Pad1.20x1.40mm_HandSolder -> Resistor_SMD:R_0805_2012Metric
- R17, R18: value 499.0K -> 240k; footprint Resistor_SMD:R_0805_2012Metric_Pad1.20x1.40mm_HandSolder -> Resistor_SMD:R_0805_2012Metric
- renumbered SW4 to SW3
Connections:
- net EN: now also J1.1 (Pin_1)
- net GND: now also J1.2 (Pin_2), J2.2 (Pin_2)
- net VBAT: now also J2.1 (Pin_1)
- net V_Input_Float: now also R21.1; no longer R17.1
- net V_Input_REF: now also R20.1; no longer R18.1
- new net: R17.1, R21.2
- new net: R18.1, R20.2
Other:
- moved on the sheet: C17, D4, D5, J10, J14, Q8, R10, R11, R14, R17, R18, R24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

Commit message: Giga Controller Updates
Parts:
- added A1: Arduino_UNO_R3, Module:Arduino_UNO_R3, symbol MCU_Module:Arduino_UNO_R3
Connections:
- net 5V-iso: no longer J10.1 (Pin_1)
- net A0: now also R11.1, A1.9 (A0)
- net A1: now also A1.10 (A1)
- net A2: now also A1.11 (A2)
- net A3: now also A1.12 (A3)
- net A4: now also A1.13 (SDA/A4)
- net A5: now also A1.14 (SCL/A5)
- net AIN3: no longer R11.1
- net D10: now also A1.25 (D10)
- net D11: now also A1.26 (D11)
- net D12: now also A1.27 (D12)
- net D13: now also A1.28 (D13)
- net D5: now also A1.20 (D5)
- net D6: now also A1.21 (D6)
- net D9: now also A1.24 (D9)
- net GND: now also J10.3 (Pin_3), A1.29 (GND), A1.6 (GND), A1.7 (GND)
- net Gnd-iso: no longer J10.3 (Pin_3)
- net RX: now also A1.15 (D0/RX)
- net SCL: now also A1.32 (SCL/A5)
- net SDA: now also A1.31 (SDA/A4)
- net TX: now also A1.16 (D1/TX)
- net USB: now also A1.5 (+5V)
- net VDD: now also J10.1 (Pin_1), A1.4 (3V3)
