File: PCBDesigns/OpenLead_Headless_V2/OpenLead_Headless_V2.kicad_pcb (KiCad board)
At the start: 4 copper layers, 23.9 x 51.3 mm, 33 parts, among them J1 Conn_01x07_Pin, J2 Battery, J3 Conn_01x07_Pin, J4 Conn_01x01, J5 Conn_01x01, J6 Conn_01x01, Q8 AO3400A MOSFET, SW3 SW_SPDT, U10 LM4040

Commit message: Working on next "Blinky Hawk" PCB version.
Parts:
- removed the J2 at (159.3, 61.7)
- removed the R14 at (158.4, 95.0)
- removed the R15 at (147.7, 75.3)
- removed SW3: SW_SPDT, Button_Switch_THT:SW_Slide_SPDT_Angled_CK_OS102011MA1Q
- added BZ1: Buzzer, Buzzer_Beeper:Buzzer_Murata_PKLCS1212E, F.Cu at (160.6, 94.7)
- added J4: Battery, Connector_PinHeader_1.27mm:PinHeader_1x02_P1.27mm_Vertical, F.Cu at (171.6, 77.6)
- added J7: Conn_01x02, Connector_PinHeader_2.54mm:PinHeader_1x02_P2.54mm_Vertical, F.Cu at (148.0, 97.8)
- added J8: Conn_01x03_Pin, Connector_PinHeader_1.27mm:PinHeader_1x03_P1.27mm_Vertical, F.Cu at (171.6, 71.0)
- added Q2: AO3400A MOSFET, Package_TO_SOT_SMD:SOT-23, F.Cu at (169.4, 96.6)
- added R17: 56K, Resistor_SMD:R_0805_2012Metric, F.Cu at (169.4, 99.8)
- added R18: 22, Resistor_SMD:R_0805_2012Metric, F.Cu at (168.2, 92.7)
- added R19: 499K, Resistor_SMD:R_0805_2012Metric, F.Cu at (152.5, 104.3)
- added R20: 499K, Resistor_SMD:R_0805_2012Metric, F.Cu at (144.8, 71.9)
- added R21: 499K, Resistor_SMD:R_0805_2012Metric, F.Cu at (146.9, 71.9)
- R16: value 1M -> 100
- R3: renamed from R29; value 100K -> 200K
- R5: renamed from R24; value 15K -> 56K
- U1: renamed from U10; value LM4040 -> LM4060 - 1.25V
- moved R16 32.9 mm to (170.5, 92.7)
- moved D1 16.7 mm to (144.9, 78.6), turned to 90 degrees
- moved D2 13.5 mm to (147.4, 78.6), turned to -90 degrees
- moved Q1 12.6 mm to (150.6, 90.4), turned to -90 degrees
- moved R8 12.5 mm to (145.5, 108.8)
- moved R5 11.9 mm to (149.6, 94.4)
- moved R4 10.4 mm to (170.5, 86.4), turned to 180 degrees
- moved R3 10.4 mm to (156.4, 104.3)
- moved R9 9.28 mm to (147.6, 110.9), turned to 90 degrees
- moved R7 8.68 mm to (145.5, 105.2), turned to 90 degrees
- moved H3 8.58 mm to (145.9, 116.2)
- moved R6 8.53 mm to (148.7, 104.3)
- moved H4 8.37 mm to (170.6, 116.2)
- moved R10 8.13 mm to (149.9, 112.8), turned to 90 degrees
- moved R11 7.59 mm to (160.2, 104.3), turned to 180 degrees
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- renumbered C17 to C1, D5 to D1, D4 to D2, J6 to J1, J5 to J2, J4 to J5, J1 to J6, Q8 to Q1, R27 to R1, R22 to R10, R17 to R11, R23 to R12, R25 to R13, R26 to R14, R28 to R15, R10 to R4, R18 to R6, R19 to R7, R20 to R8, R21 to R9
Connections:
- net SCL renamed SCL/A5
- C1 pad 1: Gnd-iso -> Gnd
- C1 pad 2: A0 -> A1
- D1 pad 2: Gnd-iso -> Gnd
- J3 pad 1: A0 -> /P014/AN09/DAC
- J3 pad 4: D3~ -> A3~
- J5 pad 1: Net-(J4-Pin_1) -> BatteryRail
- J6 pad 1: XIAO 5V -> Vbus
- J6 pad 2: Gnd-iso -> Gnd
- J6 pad 7: D7 -> Bridge_CRTL
- Q1 pad 1: A1 -> Bridge_CRTL
- R1 pad 2: A0 -> A1
- R16 pad 1: Gnd-iso -> D9~
- R16 pad 2: A0 -> Net-(Q2-G)
- R3 pad 1: A0 -> Net-(J7-Pin_1)
- R3 pad 2: Net-(R14-Pad1) (its old number) -> A2
- R4 pad 1: Gnd-iso -> Gnd
- R4 pad 2: A1 -> Bridge_CRTL
- R5 pad 2: A0 -> A1
- R6 pad 2: A0 -> A1
- U1 pad 1: A0 -> A1
- U1 pad 2: Gnd-iso -> Gnd
- U1 pad 3: Gnd-iso -> Gnd
Routing:
- net A0: track 42.6 -> 0.00 mm, vias 2 -> 0
- net Vbus: track 0.00 -> 32.3 mm
- net Net-(J2-Pin_1): track 31.2 -> 0.00 mm
- net Bridge_CRTL: track 0.00 -> 22.3 mm
- net BatteryRail: track 0.00 -> 18.7 mm
- net A1: track 28.0 -> 45.2 mm, vias 2 -> 1
- net D9~: track 0.00 -> 15.8 mm
- net Net-(BZ1--): track 0.00 -> 14.4 mm
- net Gnd: track 0.00 -> 14.0 mm, vias 0 -> 5
- net Net-(J4-Pin_1): track 13.1 -> 0.00 mm
- net Gnd-iso: track 11.7 -> 0.00 mm, vias 5 -> 0
- net Net-(J7-Pin_1): track 0.00 -> 10.8 mm
- net A3~: track 0.00 -> 7.64 mm, vias 0 -> 1
- net Net-(Q2-G): track 0.00 -> 7.36 mm
- net D10~: track 0.00 -> 6.85 mm
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- added copper zone on In1.Cu, net Gnd
- removed copper zone on In1.Cu, net Gnd-iso
Other:
- board size 23.9 x 51.3 mm -> 30 x 54.7 mm

Commit message: PCB design updates for Blinky Hawk
Parts:
- removed J7: Conn_01x02, Connector_PinHeader_2.54mm:PinHeader_1x02_P2.54mm_Vertical
- added R2: 4.7K, Resistor_SMD:R_0805_2012Metric, F.Cu at (158.0, 95.1)
- added R22: 1Meg, Resistor_SMD:R_0805_2012Metric, F.Cu at (157.9, 110.4)
- added R23: 4.7K, Resistor_SMD:R_0805_2012Metric, F.Cu at (158.0, 98.7)
- added SW1: SW_DIP_x04, Button_Switch_SMD:SW_DIP_SPSTx04_Slide_KingTek_DSHP04TS_W7.62mm_P1.27mm, F.Cu at (151.0, 105.3)
- moved R17 28.9 mm to (170.8, 70.9), turned to 0 degrees
- moved Q2 22.5 mm to (170.7, 74.1), turned to -90 degrees
- moved R4 18.8 mm to (152.0, 89.6), turned to -90 degrees
- moved R18 15.1 mm to (172.0, 78.0), turned to -90 degrees
- moved J8 15.1 mm to (171.6, 86.1)
- moved R16 14.7 mm to (169.7, 78.0), turned to 90 degrees
- moved R13 10.4 mm to (171.2, 115.4), turned to 90 degrees
- moved R12 10.1 mm to (171.2, 111.3), turned to 90 degrees
- moved R14 9.78 mm to (169.0, 117.2)
- moved R11 9.22 mm to (167.1, 110.4)
- moved R3 8.67 mm to (162.6, 110.4)
- moved R15 8.37 mm to (166.8, 119.1)
- moved J2 6.53 mm to (163.3, 120.0)
- moved H3 6.10 mm to (145.9, 122.3)
- moved H4 6.10 mm to (170.5, 122.3)
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Connections:
- J6 pad 6: D5~ -> D8
- J8 pad 2: D10~ -> D6~
- R19 pad 2: Net-(J7-Pin_1) -> Net-(R19-Pad2)
- R3 pad 1: Net-(J7-Pin_1) -> Net-(R22-Pad2)
Routing:
- net D8: track 0.00 -> 31.3 mm
- net D10~: track 6.85 -> 36.5 mm, vias 0 -> 2
- net D6~: track 0.00 -> 24.1 mm, vias 0 -> 1
- net Net-(R22-Pad2): track 0.00 -> 16.3 mm, vias 0 -> 2
- net Vbus: track 32.3 -> 45.6 mm, vias 0 -> 2
- net D9~: track 15.8 -> 4.12 mm
- net A2: track 41.8 -> 53.1 mm, vias 0 -> 2
- net Net-(J7-Pin_1): track 10.8 -> 0.00 mm
- net Net-(R19-Pad2): track 0.00 -> 9.28 mm
- net A1: track 45.2 -> 52.2 mm
- net BatteryRail: track 18.7 -> 13.9 mm
- net +3V3: track 3.97 -> 8.75 mm
- net Net-(BZ1--): track 14.4 -> 18.6 mm
- net Gnd: track 14.0 -> 16.2 mm, vias 5 -> 6
- net Net-(R11-Pad1): track 1.86 -> 3.16 mm
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Other:
- board size 30 x 54.7 mm -> 30.4 x 61.2 mm
- board text added: "OIH Designs {dblquote}Blinky Hawk{dblquote} 20260704"
- board text added: "Paired. Must Match."
- board text added: "VBus D Gnd"
- board text removed: "OIH Designs Open Lead Detect VMeter Designed 202605115"

Commit message: PCB Design Updates
Parts:
- removed U1: LM4060 - 1.25V, Package_TO_SOT_SMD:SOT-23
- added JP1: Pin2_High, Jumper:SolderJumper-2_P1.3mm_Bridged_Pad1.0x1.5mm, F.Cu at (146.8, 88.1)
- added JP2: Pin2_Gnd, Jumper:SolderJumper-2_P1.3mm_Open_TrianglePad1.0x1.5mm, F.Cu at (146.8, 90.8)
- added U3: TL431DBZ, Package_TO_SOT_SMD:SOT-23, F.Cu at (146.8, 94.1)
- BZ1: footprint Buzzer_Beeper:Buzzer_Murata_PKLCS1212E -> Buzzer_Beeper:Buzzer_12x9.5RM7.6
- moved R1 5.82 mm to (147.8, 84.7), turned to -90 degrees
- moved J5 3.43 mm to (158.6, 87.9)
- moved BZ1 3.42 mm to (162.4, 96.8)
Routing:
- net Net-(JP1-A): track 0.00 -> 6.98 mm
- net D10~: track 36.5 -> 39.5 mm
- net D6~: track 24.1 -> 26.9 mm, vias 1 -> 0
- net BatteryRail: track 13.9 -> 15.9 mm
- net Bridge_CRTL: track 21.9 -> 23.4 mm
- net Gnd: track 16.2 -> 14.8 mm, vias 6 -> 7
- net A1: track 52.2 -> 53.5 mm
- net Net-(BZ1--): track 18.6 -> 19.2 mm
- net +3V3: track 8.75 -> 8.69 mm, vias 3 -> 2
Other:
- outline, holes or cut-outs redrawn
- board text added: "Gnd"
- board text added: "Vref"
