File: PCBDesigns/OpenLead_Headless_V2/OpenLead_Headless_V2.kicad_sch (KiCad schematic)
At the start: 32 parts, among them J1 Conn_01x01, J2 Conn_01x01, J3 Conn_01x07_Pin, J4 Battery, J5 Conn_01x01, J6 Conn_01x07_Pin, Q1 AO3400A MOSFET, SW1 SW_SPDT, U1 LM4060 - 1.25V

Commit message: Working on next "Blinky Hawk" PCB version.
Parts:
- removed R2: 100K, Resistor_SMD:R_0805_2012Metric, symbol Device:R_US
- removed SW1: SW_SPDT, Button_Switch_THT:SW_Slide_SPDT_Angled_CK_OS102011MA1Q, symbol Switch:SW_SPDT
- added BZ1: Buzzer, Buzzer_Beeper:Buzzer_Murata_PKLCS1212E, symbol Device:Buzzer
- added J7: Conn_01x02, Connector_PinHeader_2.54mm:PinHeader_1x02_P2.54mm_Vertical, symbol Connector_Generic:Conn_01x02
- added J8: Conn_01x03_Pin, Connector_PinHeader_1.27mm:PinHeader_1x03_P1.27mm_Vertical, symbol Connector:Conn_01x03_Pin
- added Q2: AO3400A MOSFET, Package_TO_SOT_SMD:SOT-23, symbol Transistor_FET:DMG2302U
- added R16: 100, Resistor_SMD:R_0805_2012Metric, symbol Device:R_US
- added R17: 56K, Resistor_SMD:R_0805_2012Metric, symbol Device:R_US
- added R18: 22, Resistor_SMD:R_0805_2012Metric, symbol Device:R_US
- added R19, R20, R21: 499K, Resistor_SMD:R_0805_2012Metric, symbol Device:R_US
- J4: footprint Connector_PinSocket_2.54mm:PinSocket_1x02_P2.54mm_Vertical -> Connector_PinHeader_1.27mm:PinHeader_1x02_P1.27mm_Vertical
- R3: value 100K -> 200K
- R5: value 15K -> 56K
Connections:
- net +3V3: now also BZ1.1 (+)
- net A1: now also C1.2, R1.2, R5.2, R6.2, U1.1 (K), J7.2 (Pin_2), R19.1; no longer Q1.1 (G), R4.2
- net D10~: now also J8.2 (Pin_2)
- net D9~: now also R16.1
- net Gnd: now also J4.1 (Pin_1), J8.3 (Pin_3), Q2.2 (S), R17.1, R21.2; no longer J4.2 (Pin_2)
- net at R3.1: now also J7.1 (Pin_1), R19.2
- net BatteryRail: now reaches J5.1 (Pin_1)
- net BatteryRail: now also J4.2 (Pin_2)
- removed net A0: C1.2, J3.1 (Pin_1), R1.2, R5.2, R6.2, U1.1 (K), U2.1 (PA02_A0_D0)
- net D3~ renamed A3~
- net A3~: now also R20.1, R21.1
- net D7 renamed Bridge_CRTL
- net Bridge_CRTL: now also Q1.1 (G), R4.2
- net SCL renamed SCL/A5
- net XIAO 5V renamed Vbus
- net Vbus: now also J8.1 (Pin_1), R20.2
- new net: Q2.1 (G), R16.2, R17.2
- new net: Q2.3 (D), R18.1
- new net: BZ1.2 (-), R18.2
- new net P014/AN09/DAC: J3.1 (Pin_1), U2.1 (PA02_A0_D0)
Other:
- moved on the sheet: C1, D1, D2, J2, J3, J5, Q1, R1, R11, R12, R13, R14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

Commit message: PCB design updates for Blinky Hawk
Parts:
- removed J7: Conn_01x02, Connector_PinHeader_2.54mm:PinHeader_1x02_P2.54mm_Vertical, symbol Connector_Generic:Conn_01x02
- added R2, R23: 4.7K, Resistor_SMD:R_0805_2012Metric, symbol Device:R_US
- added R22: 1Meg, Resistor_SMD:R_0805_2012Metric, symbol Device:R_US
- added SW1: SW_DIP_x04, Button_Switch_SMD:SW_DIP_SPSTx04_Slide_KingTek_DSHP04TS_W7.62mm_P1.27mm, symbol Switch:SW_DIP_x04
Connections:
- net +3V3: now also R2.1, R23.1
- net A1: now also SW1.8
- net D10~: now also R23.2, SW1.4; no longer J8.2 (Pin_2)
- net D6~: now also J8.2 (Pin_2)
- net Gnd: now also SW1.5, SW1.6
- net at R19.2: now also R22.1, SW1.1, SW1.2; no longer R3.1
- net D5~ renamed D8
- net D8: now also R2.2, SW1.3
- new net: R22.2, R3.1, SW1.7
Other:
- moved on the sheet: C1, D1, D2, J1, J2, J3, J6, J8, Q1, R1, R10, R11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

Commit message: PCB Design Updates
Parts:
- added JP1: Pin2_High, Jumper:SolderJumper-2_P1.3mm_Bridged_Pad1.0x1.5mm, symbol Jumper:Jumper_2_Small_Bridged
- added JP2: Pin2_Gnd, Jumper:SolderJumper-2_P1.3mm_Open_TrianglePad1.0x1.5mm, symbol Jumper:Jumper_2_Small_Open
- added U3: TL431DBZ, Package_TO_SOT_SMD:SOT-23, symbol Reference_Voltage:TL431DBZ
- BZ1: footprint Buzzer_Beeper:Buzzer_Murata_PKLCS1212E -> Buzzer_Beeper:Buzzer_12x9.5RM7.6
- U1: now not fitted
Connections:
- net A1: now also JP1.2 (B), U3.1 (K); no longer U1.1 (K)
- net Gnd: now also JP2.1 (A), U3.3 (A); no longer U1.2 (A), U1.3 (nc_(gnd))
- new net: JP1.1 (A), JP2.2 (B), U3.2 (REF)
Other:
- moved on the sheet: C1, R1
