File: PCBDesigns/OpenLead_Headless_V3/OpenLead_Headless_V3.kicad_pcb (KiCad board)
At the start: 4 copper layers, 25.4 x 53.5 mm, 31 parts, among them J1 Conn_01x01, J2 Conn_01x01, J3 Conn_01x07_Pin, J4 Battery, J5 Conn_01x01, J6 Conn_01x07_Pin, Q1 AO3400A MOSFET, U3 TL431DBZ

Commit message: Blinky Hawk now has a low power sleep mode (1mA draw).
Wakes on activity, samples for activity every 1 second.

Fully configurable in the GUI.
Parts:
- added H1: MountingHole, MountingHole:MountingHole_2.2mm_M2_Pad, F.Cu at (100.8, 121.3)
- added H2: MountingHole, MountingHole:MountingHole_2.2mm_M2_Pad, F.Cu at (100.8, 127.3)
- added H3: MountingHole, MountingHole:MountingHole_2.2mm_M2_Pad, F.Cu at (100.8, 133.2)
- added H4: MountingHole, MountingHole:MountingHole_2.2mm_M2_Pad, F.Cu at (100.8, 139.2)
- added Q2: AO3400A MOSFET, Package_TO_SOT_SMD:SOT-23, F.Cu at (178.6, 94.2)
- added Q3: AO3401A, Package_TO_SOT_SMD:SOT-23, F.Cu at (178.6, 98.2)
- added R18: 100K, Resistor_SMD:R_0805_2012Metric, F.Cu at (182.8, 94.9)
- added R2: 4.7K, Resistor_SMD:R_0805_2012Metric, F.Cu at (182.8, 99.2)
- added R3: 4.7K, Resistor_SMD:R_0805_2012Metric, F.Cu at (182.8, 97.0)
- added SW1: SW_DPST, SW-TH_SS21-BBIWC2-R, F.Cu at (158.4, 119.1)
- added SW2: XY-TBT5858-W-FL, SW-SMD_6P-L5.8-W5.8-P2.00-LS11.3-1, F.Cu at (191.5, 99.1)
- moved J1 15.1 mm to (153.4, 128.8)
- moved J2 15.1 mm to (163.3, 128.8)
- moved J4 10.9 mm to (174.8, 96.5), turned to 0 degrees
Connections:
- J1 pad 1: V_Input_REF -> Net-(J1-Pin_1)
- J2 pad 1: V_Input_Float -> Net-(J2-Pin_1)
- J4 pad 2: BatteryRail -> Net-(J4-Pin_2)
Routing:
- net Net-(R18-Pad1): track 0.00 -> 10.4 mm
- net Net-(J1-Pin_1): track 0.00 -> 6.97 mm
- net Net-(Q2-G): track 0.00 -> 6.74 mm
- net Net-(J2-Pin_1): track 0.00 -> 4.87 mm
- net BatteryRail: track 20.2 -> 16.3 mm
- net Net-(Q2-D): track 0.00 -> 3.31 mm
- net V_Input_REF: track 4.05 -> 7.15 mm
- net Net-(Q3-G): track 0.00 -> 2.37 mm
Other:
- board size 25.4 x 53.5 mm -> 25.4 x 67.3 mm

Commit message: BlinkyHawk PCB V3 Firmware is now a thing
Parts:
- removed H1, H2, H3, H4: MountingHole, MountingHole:MountingHole_2.2mm_M2_Pad
- removed Q2: AO3400A MOSFET, Package_TO_SOT_SMD:SOT-23
- removed Q3: AO3401A, Package_TO_SOT_SMD:SOT-23
- removed R18: 100K, Resistor_SMD:R_0805_2012Metric
- removed R2, R3: 4.7K, Resistor_SMD:R_0805_2012Metric
- removed SW1: SW_DPST, SW-TH_SS21-BBIWC2-R
- removed SW2: XY-TBT5858-W-FL, SW-SMD_6P-L5.8-W5.8-P2.00-LS11.3-1
- J1, J2: footprint Connector_Wire:SolderWire-0.75sqmm_1x01_D1.25mm_OD2.3mm -> Connector_Wire:SolderWirePad_1x01_SMD_1.5x3mm
- R20, R21: value 499K -> 100K
- moved J2 17.8 mm to (162.1, 111.0), turned to 180 degrees
- moved J1 17.8 mm to (153.4, 111.0), turned to 180 degrees
- moved J4 9.48 mm to (169.3, 88.8)
- moved R1 6.74 mm to (147.1, 95.1)
- moved LED1 0.34 mm to (169.4, 94.6), turned to 90 degrees
Connections:
- J1 pad 1: Net-(J1-Pin_1) -> V_Input_REF
- J2 pad 1: Net-(J2-Pin_1) -> V_Input_Float
- J4 pad 2: Net-(J4-Pin_2) -> BatteryRail
Routing:
- net Net-(R18-Pad1): track 10.4 -> 0.00 mm
- net Net-(J1-Pin_1): track 6.97 -> 0.00 mm
- net Net-(Q2-G): track 6.74 -> 0.00 mm
- net Net-(U3-K): track 25.4 -> 18.9 mm
- net Net-(J2-Pin_1): track 4.87 -> 0.00 mm
- net V_Input_REF: track 7.15 -> 3.00 mm
- net Net-(BZ1-+): track 15.5 -> 12.0 mm
- net Net-(Q2-D): track 3.31 -> 0.00 mm
- net BatteryRail: track 16.3 -> 19.0 mm, vias 1 -> 0
- net Net-(Q3-G): track 2.37 -> 0.00 mm
- net V_Input_Float: track 6.22 -> 4.16 mm
- net +3V3: track 2.58 -> 4.08 mm, vias 2 -> 1
- net D6~: track 25.1 -> 26.2 mm
- net Net-(BZ1--): vias 0 -> 2
Other:
- board size 25.4 x 67.3 mm -> 25.4 x 51.9 mm
