File: PCBDesigns/BlinkyHawk_V3b/BlinkyHawk_V3b.kicad_pcb (KiCad board)
At the start: 4 copper layers, 25.4 x 51.9 mm, 29 parts, among them J1 Conn_01x01, J2 Conn_01x01, J3 Conn_01x07_Pin, J4 Battery, J5 Conn_01x01, J6 Conn_01x07_Pin, Q1 AO3400A MOSFET, U3 TL431DBZ

Commit message: Working on next BlinkyHawk PCB
Parts:
- added C10: 0.1uF, Capacitor_SMD:C_0402_1005Metric, F.Cu at (167.4, 75.0)
- added C2: 0.47uF, Capacitor_SMD:C_0402_1005Metric, F.Cu at (148.0, 86.6)
- added C3: 1uF, Capacitor_SMD:C_0402_1005Metric, F.Cu at (185.1, 87.2)
- added C4: 1uF, Capacitor_SMD:C_0402_1005Metric, F.Cu at (181.3, 87.2)
- added C5: 2.2uF, Capacitor_SMD:C_0402_1005Metric, F.Cu at (179.6, 89.6)
- added C6: 2.2uF, Capacitor_SMD:C_0402_1005Metric, F.Cu at (179.6, 91.8)
- added C7: 1uF, Capacitor_SMD:C_0402_1005Metric, F.Cu at (148.1, 75.7)
- added C8: 1uF, Capacitor_SMD:C_0402_1005Metric, F.Cu at (166.1, 74.0)
- added C9: 0.1uF, Capacitor_SMD:C_0402_1005Metric, F.Cu at (148.0, 73.3)
- added J7: Conn_01x01, TestPoint:TestPoint_Pad_1.0x1.0mm, B.Cu at (163.3, 74.0)
- added U1: TPS22914BYFPR, easyeda_parts:DSBGA-4_L0.8-W0.8-R2-C2-P0.40-BL, F.Cu at (148.3, 74.2)
- added U4: TPS22914BYFPR, easyeda_parts:DSBGA-4_L0.8-W0.8-R2-C2-P0.40-BL, F.Cu at (167.3, 73.5)
- added U5: PAM8904JER, easyeda_parts:TQFN-16_L3.0-W3.0-P0.50-BL-EP1.5, F.Cu at (183.5, 90.4)
- C1: footprint Capacitor_SMD:C_0805_2012Metric -> Capacitor_SMD:C_0402_1005Metric
- J5: footprint Connector_Wire:SolderWire-0.5sqmm_1x01_D0.9mm_OD2.1mm -> TestPoint:TestPoint_Pad_1.0x1.0mm; moved to B.Cu
- LED1: footprint LED_SMD:LED-SMD_4P-L4.0-W1.6-L -> easyeda_parts:LED-SMD_4P-L4.0-W1.6-L
- moved J5 13.8 mm to (158.9, 74.0)
- moved R20 13.7 mm to (147.2, 60.1)
- moved J3 13.7 mm to (151.0, 54.0)
- moved J6 13.7 mm to (166.2, 54.0)
- moved R21 13.7 mm to (147.2, 63.9)
Connections:
- BZ1 pad 1: D8 -> Net-(BZ1-+)
- BZ1 pad 2: D9 -> Net-(BZ1--)
- LED1 pad 2: BatteryRail -> LEDRail
- R1 pad 1: +3V3 -> Analog_Rail
Routing:
- net D8: track 17.0 -> 6.43 mm
- net BatteryRail: track 19.0 -> 8.58 mm
- net D9: track 29.7 -> 22.7 mm
- net Net-(U5-CP2): track 0.00 -> 6.05 mm
- net Net-(U5-CN1): track 0.00 -> 5.78 mm
- net A2: track 39.8 -> 36.8 mm
- net Net-(U5-CN2): track 0.00 -> 2.50 mm
- net Net-(BZ1-+): track 0.00 -> 1.78 mm
- net LEDRail: track 0.00 -> 1.68 mm
- net Net-(U5-VOUT): track 0.00 -> 1.53 mm
- net Bridge_CRTL: track 21.5 -> 20.8 mm
- net +3V3: track 4.08 -> 3.44 mm
Other:
- board size 25.4 x 51.9 mm -> 25.4 x 65.7 mm
- board text added: "D15"

Commit message: Next BlinkyHawk PCB Work
Parts:
- removed D1, D2: D_Schottky, Diode_SMD:D_SOD-123
- added D3: BAT54S, Package_TO_SOT_SMD:SOT-23, F.Cu at (150.5, 91.3)
- BZ1: footprint Buzzer_Beeper:Buzzer_Murata_PKLCS1212E -> easyeda_parts:BUZ-SMD_2P-L12.0-W12.0-L_PKLCS1212E4001-R1
- moved C10 26.0 mm to (169.7, 100.9)
- moved C3 25.9 mm to (159.3, 87.4), turned to 90 degrees
- moved U4 25.8 mm to (169.6, 99.2)
- moved C8 25.8 mm to (168.1, 99.8)
- moved U5 21.9 mm to (162.1, 85.8), turned to 180 degrees
- moved C4 17.0 mm to (164.3, 88.4), turned to 180 degrees
- moved C9 15.2 mm to (149.1, 88.4), turned to 180 degrees
- moved C6 15.0 mm to (166.1, 85.1), turned to 0 degrees
- moved C5 14.8 mm to (165.1, 86.6), turned to 0 degrees
- moved U1 14.3 mm to (147.4, 88.5)
- moved J4 14.0 mm to (155.4, 86.7)
- moved C7 13.9 mm to (147.1, 89.5), turned to 0 degrees
- moved J5 10.7 mm to (158.9, 84.7)
- moved J7 10.7 mm to (163.3, 84.7)
- moved R20 10.7 mm to (147.2, 70.7)
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Connections:
- C7 pad 2: unconnected-(C7-Pad2) -> Gnd
- C9 pad 1: unconnected-(C9-Pad1) -> Gnd
- R20 pad 1: A3 -> A1
- R21 pad 1: A3 -> A1
- U1 pad B2: A1 -> A3
Routing:
- net BatteryRail: track 8.58 -> 40.0 mm, vias 0 -> 3
- net D10: track 0.00 -> 29.9 mm, vias 0 -> 1
- net Net-(BZ1--): track 0.00 -> 16.9 mm, vias 0 -> 2
- net A3: track 6.05 -> 19.0 mm
- net Gnd: track 8.49 -> 19.0 mm, vias 6 -> 14
- net Analog_Rail: track 0.00 -> 9.89 mm
- net D9: track 22.7 -> 14.0 mm, vias 2 -> 1
- net A1: track 0.00 -> 8.26 mm
- net D8: track 6.43 -> 13.1 mm
- net LEDRail: track 1.68 -> 8.26 mm, vias 0 -> 2
- net Bridge_CRTL: track 20.8 -> 26.1 mm, vias 0 -> 1
- net A2: track 36.8 -> 42.1 mm
- net D15: track 0.00 -> 4.79 mm, vias 0 -> 1
- net Net-(U5-CP1): track 0.00 -> 4.70 mm, vias 0 -> 2
- net D6: track 26.2 -> 29.9 mm, vias 1 -> 3
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Other:
- board size 25.4 x 65.7 mm -> 25.4 x 55 mm

Commit message: AD8237DevBoardTestDesign
Parts:
- removed J3, J6: Conn_01x07_Pin, Connector_PinSocket_2.54mm:PinSocket_1x07_P2.54mm_Vertical
- added U2: ~, Seeed_XIAO:XIAO-R4-DIP, F.Cu at (158.6, 73.3)
- C2: value 0.47uF -> 1uF
- moved J5 1.88 mm to (158.0, 86.4)
- moved C4 1.04 mm to (164.3, 89.4)
- moved C3 1.04 mm to (159.3, 88.4)
- moved C5 1.04 mm to (165.1, 87.7)
- moved C6 1.04 mm to (166.1, 86.1)
- moved J7 1.04 mm to (163.3, 85.7)
- moved U5 1.04 mm to (162.1, 86.9)
- moved R20 1.02 mm to (147.2, 71.8)
- moved R21 1.02 mm to (147.2, 75.6)
- moved J4 0.13 mm to (155.4, 86.6)
Routing:
- net BatteryRail: track 40.0 -> 37.0 mm
- net D6: track 29.9 -> 28.8 mm
- net Net-(BZ1--): track 16.9 -> 15.8 mm
- net A3: track 19.0 -> 18.0 mm
- net A2: track 42.1 -> 41.1 mm
- net D10: track 29.9 -> 28.9 mm
- net Net-(BZ1-+): track 3.19 -> 2.50 mm
- net D8: track 13.1 -> 12.6 mm
Other:
- board size 25.4 x 55 mm -> 25.4 x 53.3 mm
- board text added: "OIH Designs {dblquote}Blinky Hawk{dblquote} 20260916"
- board text removed: "OIH Designs {dblquote}Blinky Hawk{dblquote} 20260801"
