File: PCBDesigns/BlinkyHawk_V3b/BlinkyHawk_V3b.kicad_sch (KiCad schematic)
At the start: 38 parts, among them J1 Conn_01x01, J2 Conn_01x01, J3 Conn_01x07_Pin, J4 Battery, J5 Conn_01x01, J6 Conn_01x07_Pin, Q1 AO3400A MOSFET, Q2 AO3400A MOSFET, Q3 AO3401A, SW2 XY-TBT5858-W-FL, SW3 SW_Toggle_3PDT, U3 TL431DBZ

Commit message: Next BlinkyHawk PCB Work
Parts:
- removed D1, D2: D_Schottky, Diode_SMD:D_SOD-123, symbol Device:D_Schottky
- added C10, C9: 0.1uF, Capacitor_SMD:C_0402_1005Metric, symbol Device:C
- added C2: 0.47uF, Capacitor_SMD:C_0402_1005Metric, symbol Device:C
- added C3, C4, C7, C8: 1uF, Capacitor_SMD:C_0402_1005Metric, symbol Device:C
- added C5, C6: 2.2uF, Capacitor_SMD:C_0402_1005Metric, symbol Device:C
- added D3: BAT54S, Package_TO_SOT_SMD:SOT-23, symbol Diode:BAT54S
- added J7: Conn_01x01, TestPoint:TestPoint_Pad_1.0x1.0mm, symbol Connector_Generic:Conn_01x01
- added U1, U4: TPS22914BYFPR, easyeda_parts:DSBGA-4_L0.8-W0.8-R2-C2-P0.40-BL, symbol easyeda_parts:TPS22914BYFPR
- added U5: PAM8904JER, easyeda_parts:TQFN-16_L3.0-W3.0-P0.50-BL-EP1.5, symbol easyeda_parts:PAM8904JER
- BZ1: footprint Buzzer_Beeper:Buzzer_Murata_PKLCS1212E -> easyeda_parts:BUZ-SMD_2P-L12.0-W12.0-L_PKLCS1212E4001-R1
- C1: footprint Capacitor_SMD:C_0805_2012Metric -> Capacitor_SMD:C_0402_1005Metric
- J5: footprint Connector_Wire:SolderWire-0.5sqmm_1x01_D0.9mm_OD2.1mm -> TestPoint:TestPoint_Pad_1.0x1.0mm
- U2: now fitted
Connections:
- net +3V3: now also C6.1, U5.15 (VIN); no longer R1.1
- net A1: now also R20.1, R21.1
- net A2: now also D3.3 (COM)
- net A3: now also U1.B2 (ON); no longer R20.1, R21.1
- net BatteryRail: now also C7.1, C8.1, D3.2 (K), U1.A2 (VIN), U4.A2 (VIN); no longer LED1.2 (VDD)
- net D10: now also U4.B2 (ON)
- net D8: now also U5.1 (EN1); no longer BZ1.1 (+)
- net D9: now also U5.2 (EN2); no longer BZ1.2 (-)
- net Gnd: now also C10.1, C2.1, C5.2, C6.2, C7.2, C8.2, C9.1, D3.1 (A), U1.B1 (GND), U4.B1 (GND), U5.6 (GND)
- new net: BZ1.1 (+), U5.9 (VO1)
- new net: BZ1.2 (-), U5.7 (VO2)
- new net: C5.1, U5.13 (VOUT)
- new net: C4.2, U5.10 (CN2)
- new net: C3.1, U5.11 (CP1)
- new net: C4.1, U5.14 (CP2)
- new net: C3.2, U5.5 (CN1)
- new net Analog_Rail: C2.2, C9.2, R1.1, U1.A1 (VOUT)
- new net D15: J7.1 (Pin_1), U5.3 (DIN)
- new net LEDRail: C10.2, LED1.2 (VDD), U4.A1 (VOUT)
Other:
- moved on the sheet: BZ1, C1, R1

Commit message: AD8237DevBoardTestDesign
Parts:
- C2: value 0.47uF -> 1uF
- U2: footprint (none) -> Seeed_XIAO:XIAO-R4-DIP
Changed lines of the file:
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@@
 		(exclude_from_sim no)
 		(in_bom yes)
-		(on_board yes)
+		(on_board no)
 		(in_pos_files yes)
 		(dnp yes)
@@
 			)
 		)
-		(property "Footprint" ""
+		(property "Footprint" "Seeed_XIAO:XIAO-R4-DIP"
 			(at 215.9 40.64 0)
 			(hide yes)
@@
 		(exclude_from_sim no)
 		(in_bom yes)
-		(on_board yes)
+		(on_board no)
 		(in_pos_files yes)
 		(dnp yes)
@@
 			)
 		)
-		(property "Value" "0.47uF"
+		(property "Value" "1uF"
 			(at 27.432 149.098 0)
 			(show_name no)
