File: PCBDesigns/BlinkyHawk_V4/BlinkyHawk_V4.kicad_pcb (KiCad board)
At the start: 4 copper layers, 25.4 x 53.3 mm, 40 parts, among them J1 Conn_01x01, J2 Conn_01x01, J4 Battery, J5 Conn_01x01, J7 Conn_01x01, Q1 AO3400A MOSFET, U1 TPS22914BYFPR, U3 TL431DBZ, U4 TPS22914BYFPR, U5 PAM8904JER

Commit message: Test Suite Updates and Data Collected
Parts:
- removed J1, J2: Conn_01x01, Connector_Wire:SolderWirePad_1x01_SMD_1.5x3mm
- added C15: 4.7uF, Capacitor_SMD:C_0805_2012Metric_Pad1.18x1.45mm_HandSolder, F.Cu at (129.8, 93.5)
- added C16: 22uF, Capacitor_SMD:C_0805_2012Metric_Pad1.18x1.45mm_HandSolder, F.Cu at (128.7, 84.8)
- added C19: 22uF, Capacitor_SMD:C_0805_2012Metric_Pad1.18x1.45mm_HandSolder, F.Cu at (128.7, 82.0)
- added L1: 2.2uH, Inductor_SMD:L_Murata_DFE201610P, F.Cu at (128.5, 91.0)
- added R16: 100K, Resistor_SMD:R_1206_3216Metric, F.Cu at (167.8, 118.0)
- added SW1: SW_Push_DPDT, Button_Switch_THT:SW_PUSH_E-Switch_FS5700DP_DPDT, F.Cu at (162.1, 120.4)
- added SW4: SW_SPDT, Button_Switch_THT:SW_Slide_SPDT_Angled_CK_OS102011MA1Q, F.Cu at (119.5, 88.1)
- added U9: TPS613222ADBV, Package_TO_SOT_SMD:SOT-23-5, F.Cu at (128.5, 87.8)
Connections:
- C7 pad 1: BatteryRail -> 5vRail
- C8 pad 1: BatteryRail -> 5vRail
- D3 pad 2: BatteryRail -> 5vRail
- R20 pad 2: Vbus -> 5vRail
- U1 pad A2: BatteryRail -> 5vRail
- U2 pad 14: Vbus -> 5vRail
- U4 pad A2: BatteryRail -> 5vRail
Routing:
- net 5vRail: track 0.00 -> 32.5 mm
- net Vbus: track 26.0 -> 0.00 mm
- net V_Input_Float: track 4.16 -> 26.0 mm, vias 0 -> 1
- net Net-(R16-Pad2): track 0.00 -> 6.75 mm
- net Net-(R16-Pad1): track 0.00 -> 5.89 mm
- net V_Input_REF: track 3.00 -> 7.74 mm
- net Net-(U9-SW): track 0.00 -> 1.97 mm
- net Net-(SW4-B): track 0.00 -> 1.58 mm
- net GND: vias 0 -> 1
- added copper zone on F.Cu, net 5vRail
- added copper zone on F.Cu, net GND
- added copper zone on F.Cu, net Net-(SW4-B)
- added copper zone on F.Cu, net Net-(U9-SW)
Other:
- board size 25.4 x 53.3 mm -> 25.4 x 61.8 mm

Commit message: 120V Monitor Updates
Parts:
- removed C15: 4.7uF, Capacitor_SMD:C_0805_2012Metric_Pad1.18x1.45mm_HandSolder
- removed C16, C19: 22uF, Capacitor_SMD:C_0805_2012Metric_Pad1.18x1.45mm_HandSolder
- removed L1: 2.2uH, Inductor_SMD:L_Murata_DFE201610P
- removed U9: TPS613222ADBV, Package_TO_SOT_SMD:SOT-23-5
- J4: footprint Connector_PinHeader_1.27mm:PinHeader_1x02_P1.27mm_Vertical -> Connector_Molex:Molex_PicoBlade_53398-0271_1x02-1MP_P1.25mm_Vertical
- moved J4 18.4 mm to (137.0, 87.0), turned to 180 degrees
- moved SW4 16.9 mm to (134.6, 95.7)
Connections:
- J4 pad 2: BatteryRail -> Net-(J4-Pin_2)
- J5 pad 1: BatteryRail -> Net-(J5-Pin_1)
- SW4 pad 1: BatteryRail -> Net-(J4-Pin_2)
- SW4 pad 2: Net-(SW4-B) -> Net-(J5-Pin_1)
Routing:
- net BatteryRail: track 37.0 -> 0.00 mm, vias 3 -> 0
- net 5vRail: track 32.5 -> 62.9 mm, vias 0 -> 3
- net Net-(U9-SW): track 1.97 -> 0.00 mm
- net Net-(SW4-B): track 1.58 -> 0.00 mm
- net GND: vias 1 -> 0
- removed copper zone on F.Cu, net 5vRail
- removed copper zone on F.Cu, net GND
- removed copper zone on F.Cu, net Net-(SW4-B)
- removed copper zone on F.Cu, net Net-(U9-SW)
